File: pcb/temper_optimized_hq.kicad_pcb (KiCad board)
At the start: 4 copper layers, 100 x 150 mm, 33 parts, among them Q1 IKW40N120H3, Q2 IKW40N120H3

Commit message: feat(routing): Complete router improvement work with comprehensive TDD test suite
## Summary
- Fixed GradNorm bug in placement optimizer
- Completed quality improvement analysis (26% routing, 854 DRC violations)
- Created router improvement epics (temper-308j, temper-su6u)
- Wrote comprehensive TDD/BDD test suite (1680+ tests)

## Router Quality Improvements (temper-308j)
- 5 tasks for immediate MazeRouter improvements
- BDD specs for blocking behavior
- Configurable margins, layer-specific blocking
- Enhanced escape routes

## Push-and-Shove Router (temper-su6u)
- 14 tasks for production-quality router
- Functional architecture with pure primitives
- Immutable Path with SDF collision detection
- Full property-based testing

## Test Suite (1680+ tests)
- Metamorphic testing (500+ tests)
- Contract-based testing (300+ tests)
- Mutation testing (verifies tests catch bugs)
- Fuzzing (1000+ random inputs)
- Real-world scenarios (power supply, BGA, differential pairs)
- Performance benchmarks

## Files Changed
- Added comprehensive test suite in tests/routing/
- Fixed optimizer/train.py GradNorm bug
- Removed deprecated FreeRouting code
- Added trace_writer.py and internal_route.py
- Updated documentation

All tests emphasize TDD/BDD, DRY, verifiability, elegance, and functional composition.
Parts:
- moved MH3 59.4 mm to (30.6, 75.0)
- moved MH1 20.0 mm to (90.0, 75.0)
- moved MH2 20.0 mm to (70.0, 75.0)
- moved MH4 19.4 mm to (50.0, 75.0)
Changed lines of the file:
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@@
   )
   (footprint "MountingHole:MountingHole_3.2mm_M3" (layer "F.Cu")
-    (at 70.0 75.0 180.0)
+    (at 90.0 75.0 180.0)
     (property "Reference" "MH1")
     (property "Value" "MountingHole_3.2mm_M3")
@@
   )
   (footprint "MountingHole:MountingHole_3.2mm_M3" (layer "F.Cu")
-    (at 50.0 75.0 90.0)
+    (at 70.0 75.0 90.0)
     (property "Reference" "MH2")
     (property "Value" "MountingHole_3.2mm_M3")
@@
   )
   (footprint "MountingHole:MountingHole_3.2mm_M3" (layer "F.Cu")
-    (at 90.0 75.0 270.0)
+    (at 30.634014129638672 75.0 270.0)
     (property "Reference" "MH3")
     (property "Value" "MountingHole_3.2mm_M3")
@@
   )
   (footprint "MountingHole:MountingHole_3.2mm_M3" (layer "F.Cu")
-    (at 30.634014129638672 75.0 90.0)
+    (at 50.0 75.0 90.0)
     (property "Reference" "MH4")
     (property "Value" "MountingHole_3.2mm_M3")
