File: pcb/power_management.kicad_sch (KiCad schematic)
At the start: 11 parts

Commit message: fix: repair schematic wiring across all six PCB sheets
Systematic audit-and-verify pass over pcb/*.kicad_sch using a custom
union-find connectivity tracer, since KiCad's own ERC/netlist export only
confirm a file parses, not that intended nets are correct.

Found and fixed several serious latent bugs, none caught by prior tooling:
- mcu.kicad_sch: +3.3V shorted to two GPIOs; RTD_CS wired to the reset pin
  instead of a GPIO; all digital pins realigned to firmware/temper_pins.h
  after verifying firmware's pin choices against the real module symbol.
- half_bridge.kicad_sch: high-side IGBT wired backwards; bootstrap diode
  backwards; UCC21550 gate driver's entire control/supply side unwired.
- safety_interlock.kicad_sch: OCP comparator inputs swapped (inverted
  fault polarity); systematic wire-gap bug across comparators/logic gates;
  full NAND SR-latch rebuilt using real datasheet pin maps recovered from
  KiCad's own bundled multi-unit symbol libraries.
- power_management.kicad_sch: buck converter's SW pin was wired into the
  feedback divider instead of FB (coordinate typo); both ICs fully wired.
- power_input.kicad_sch: both mains rectifier diodes (D1, D2) in the
  voltage-doubler stage installed backwards, resolved via independent
  circuit-theory verification after design doc and atopile source
  disagreed with each other.
- sensing.kicad_sch: parse-blocking symbol bug; MAX31865 and ADUM1250
  fully wired (both were 100% unconnected).

user_interface.kicad_sch required no changes - confirmed already correct.

Documented the reusable techniques and root causes in docs/solutions/.

Co-Authored-By: Claude Sonnet 5 <noreply@anthropic.com>
Connections:
- net +3.3V is gone; now on net GND: C_OUT_LDO.1
- net DC_BUS+: now also C_BOOT_BUCK.2, L_BUCK.1
- net GND: now also U_LDO.3 (CE)
Changed lines of the file:
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@@
   )
   (wire
-    (pts (xy 114.3 93.98) (xy 121.92 93.98))
+    (pts (xy 114.3 83.82) (xy 121.92 83.82))
     (stroke (width 0) (type default))
     (uuid "wire-fb-pin-001")
   )
   (wire
-    (pts (xy 121.92 93.98) (xy 121.92 97.79))
+    (pts (xy 121.92 83.82) (xy 121.92 97.79))
     (stroke (width 0) (type default))
     (uuid "wire-fb-pin-002")
@@
     (uuid "text-ldo-notes-001")
   )
+  (wire (pts (xy 88.9 93.98) (xy 10.0 93.98)) (stroke (width 0) (type default)))
+  (wire (pts (xy 10.0 93.98) (xy 10.0 200.0)) (stroke (width 0) (type default)))
+  (wire (pts (xy 25.4 88.9) (xy 10.0 88.9)) (stroke (width 0) (type default)))
+  (wire (pts (xy 10.0 88.9) (xy 10.0 200.0)) (stroke (width 0) (type default)))
+  (wire (pts (xy 88.9 88.9) (xy 11.4 88.9)) (stroke (width 0) (type default)))
+  (wire (pts (xy 11.4 88.9) (xy 11.4 202.0)) (stroke (width 0) (type default)))
+  (wire (pts (xy 25.4 88.9) (xy 11.4 88.9)) (stroke (width 0) (type default)))
+  (wire (pts (xy 11.4 88.9) (xy 11.4 202.0)) (stroke (width 0) (type default)))
+  (wire (pts (xy 101.6 78.74) (xy 12.8 78.74)) (stroke (width 0) (type default)))
+  (wire (pts (xy 12.8 78.74) (xy 12.8 204.0)) (stroke (width 0) (type default)))
+  (wire (pts (xy 25.4 127.0) (xy 12.8 127.0)) (stroke (width 0) (type default)))
+  (wire (pts (xy 12.8 127.0) (xy 12.8 204.0)) (stroke (width 0) (type default)))
+  (wire (pts (xy 114.3 93.98) (xy 14.2 93.98)) (stroke (width 0) (type default)))
+  (wire (pts (xy 14.2 93.98) (xy 14.2 206.0)) (stroke (width 0) (type default)))
+  (wire (pts (xy 135.89 76.2) (xy 14.2 76.2)) (stroke (width 0) (type default)))
+  (wire (pts (xy 14.2 76.2) (xy 14.2 206.0)) (stroke (width 0) (type default)))
+  (wire (pts (xy 157.48 154.94) (xy 15.6 154.94)) (stroke (width 0) (type default)))
+  (wire (pts (xy 15.6 154.94) (xy 15.6 208.0)) (stroke (width 0) (type default)))
+  (wire (pts (xy 152.4 152.4) (xy 15.6 152.4)) (stroke (width 0) (type default)))
+  (wire (pts (xy 15.6 152.4) (xy 15.6 208.0)) (stroke (width 0) (type default)))
+  (wire (pts (xy 157.48 152.4) (xy 17.0 152.4)) (stroke (width 0) (type default)))
+  (wire (pts (xy 17.0 152.4) (xy 17.0 210.0)) (stroke (width 0) (type default)))
+  (wire (pts (xy 157.48 154.94) (xy 17.0 154.94)) (stroke (width 0) (type default)))
+  (wire (pts (xy 17.0 154.94) (xy 17.0 210.0)) (stroke (width 0) (type default)))
+  (wire (pts (xy 165.1 144.78) (xy 18.4 144.78)) (stroke (width 0) (type default)))
+  (wire (pts (xy 18.4 144.78) (xy 18.4 212.0)) (stroke (width 0) (type default)))
+  (wire (pts (xy 25.4 127.0) (xy 18.4 127.0)) (stroke (width 0) (type default)))
+  (wire (pts (xy 18.4 127.0) (xy 18.4 212.0)) (stroke (width 0) (type default)))
+  (wire (pts (xy 172.72 154.94) (xy 19.8 154.94)) (stroke (width 0) (type default)))
+  (wire (pts (xy 19.8 154.94) (xy 19.8 214.0)) (stroke (width 0) (type default)))
+  (wire (pts (xy 228.6 152.4) (xy 19.8 152.4)) (stroke (width 0) (type default)))
+  (wire (pts (xy 19.8 152.4) (xy 19.8 214.0)) (stroke (width 0) (type default)))
 )
