File: pcb/power_management.kicad_sch (KiCad schematic)
At the start: 13 parts, among them U3 LMR51430XDDCR

Commit message: fix(hardware): float SELV control domain, remove star-point ground join
Removes `power_return ~ gnd`, which shorted the AuxSupply IRM-10-15's
4.2kVAC isolation barrier by making the SELV control-domain ground the
same net as the HV doubler midpoint (which tracks AC Neutral). SELV
ground is now bonded directly to protective earth instead, reusing the
existing Y1-cap PE bond point on the HV side without disturbing it.

Isolates the zero-crossing-detect signal with a new H11L1 optocoupler
(verified datasheet pinout/ratings), resolving the project's own
pre-existing TODO. Corrects the "+340V_BUS" net name/comment on
dc_bus_plus, which is actually the +170V half-bus of the Delon doubler
-- that wrong name is what would cause OVP-01's reference divider to be
mistuned by 2x if someone trusted it over the topology; OVPComparator's
docstring now carries the derivation and a warning against that.
Updates RTDSensing's docstring to state what is actually true post-fix
rather than an unqualified isolation claim the netlist didn't fully
support.

Full crossing survey, falsifier result, netlist evidence that gnd and
PWR_RTN are now separate nets, ERC results, and ranked open items
(principally: the OVP-01 bus-sense divider still bridges HV into gnd
resistively and needs a separate part addition to isolate) are in
docs/hardware/SELV_ISOLATION_REDESIGN.md.

Co-Authored-By: Claude Opus 5 <noreply@anthropic.com>
Parts:
- renumbered R19 to R21, R20 to R22, U3 to U4
Connections:
- net PWR_RTN: no longer C11.2, C12.2, C13.2, C15.2, C16.2, C9.2, PS1.4, R22.2, U4.1
- net +340V_BUS renamed +170V_BUS
- new net gnd: C11.2, C12.2, C13.2, C15.2, C16.2, C9.2, PS1.4, R22.2, U4.1
Changed lines of the file:
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@@
     (effects (font (size 1.27 1.27)) (justify left bottom))
   )
-  (hierarchical_label "PWR_RTN"
+  (hierarchical_label "gnd"
     (shape bidirectional)
     (at 106.04 50.80 0)
@@
     (effects (font (size 1.27 1.27)) (justify left bottom))
   )
-  (hierarchical_label "PWR_RTN"
+  (hierarchical_label "gnd"
     (shape bidirectional)
     (at 146.04 50.80 0)
@@
     (effects (font (size 1.27 1.27)) (justify left bottom))
   )
-  (hierarchical_label "PWR_RTN"
+  (hierarchical_label "gnd"
     (shape bidirectional)
     (at 186.04 50.80 0)
@@
     (pin "2")
   )
-  (hierarchical_label "+340V_BUS"
+  (hierarchical_label "+170V_BUS"
     (shape bidirectional)
     (at 195.56 50.80 0)
@@
     (effects (font (size 1.27 1.27)) (justify left bottom))
   )
-  (hierarchical_label "PWR_RTN"
+  (hierarchical_label "gnd"
     (shape bidirectional)
     (at 66.04 80.80 0)
@@
     (effects (font (size 1.27 1.27)) (justify left bottom))
   )
-  (hierarchical_label "PWR_RTN"
+  (hierarchical_label "gnd"
     (shape bidirectional)
     (at 106.04 80.80 0)
@@
     (effects (font (size 1.27 1.27)) (justify left bottom))
   )
-  (hierarchical_label "PWR_RTN"
+  (hierarchical_label "gnd"
     (shape bidirectional)
     (at 146.04 80.80 0)
@@
     (pin "4")
   )
-  (hierarchical_label "+340V_BUS"
+  (hierarchical_label "+170V_BUS"
     (shape bidirectional)
     (at 195.56 83.34 0)
@@
     (effects (font (size 1.27 1.27)) (justify left bottom))
   )
-  (hierarchical_label "PWR_RTN"
+  (hierarchical_label "gnd"
     (shape bidirectional)
     (at 226.04 78.26 0)
@@
     (on_board yes)
     (dnp no)
-    (property "Reference" "R19" (at 50.80 108.26 0) (effects (font (size 1.27 1.27))))
+    (property "Reference" "R21" (at 50.80 108.26 0) (effects (font (size 1.27 1.27))))
     (property "Value" "RC0603FR-0710KL" (at 50.80 113.34 0) (effects (font (size 1.27 1.27))))
     (property "Footprint" "Resistor_SMD:R_0603_1608Metric" (at 50.80 110.80 0) (effects (font (size 1.27 1.27)) hide))
@@
     (on_board yes)
     (dnp no)
-    (property "Reference" "R20" (at 90.80 108.26 0) (effects (font (size 1.27 1.27))))
+    (property "Reference" "R22" (at 90.80 108.26 0) (effects (font (size 1.27 1.27))))
     (property "Value" "RC0603FR-0710KL" (at 90.80 113.34 0) (effects (font (size 1.27 1.27))))
     (property "Footprint" "Resistor_SMD:R_0603_1608Metric" (at 90.80 110.80 0) (effects (font (size 1.27 1.27)) hide))
@@
     (effects (font (size 1.27 1.27)) (justify left bottom))
   )
-  (hierarchical_label "PWR_RTN"
+  (hierarchical_label "gnd"
     (shape bidirectional)
     (at 106.04 110.80 0)
@@
     (on_board yes)
     (dnp no)
-    (property "Reference" "U3" (at 130.80 108.26 0) (effects (font (size 1.27 1.27))))
+    (property "Reference" "U4" (at 130.80 108.26 0) (effects (font (size 1.27 1.27))))
     (property "Value" "LMR51430XDDCR" (at 130.80 113.34 0) (effects (font (size 1.27 1.27))))
     (property "Footprint" "Package_TO_SOT_SMD:SOT-23-6" (at 130.80 110.80 0) (effects (font (size 1.27 1.27)) hide))
@@
     (pin "6")
   )
-  (hierarchical_label "PWR_RTN"
+  (hierarchical_label "gnd"
     (shape bidirectional)
     (at 115.56 115.88 0)

Commit message: fix(hardware): re-verify SELV isolation redesign after rebase
Rebases the SELV-float change onto the current tip of
docs/methodology-loop-discipline, which had moved ahead by several
commits (THM-02, OCP-02, UVL-02, and BOM part-number replacements) since
the worktree this was originally built in was created. Re-derives every
finding against the rebased tree rather than carrying the old ones
forward:

- OVP-01 conclusion corrected: the rebased tree's OVPComparator carries
  r_ref_top=1.1k/r_hyst=287k (not the 12k/no-hysteresis value the stale
  worktree had), which trips at ~400V on a node (dc_bus_plus) that can
  only reach ~170-250V -- OVP-01 is fail-open, matching
  docs/STRATEGY.md's independently-landed "OVP-01 is fail-open" entry.
  Not re-tuned here; flagged with two remediation options and a
  recommendation.
- Crossing survey extended for the three modules that landed on the
  rebase: CoilThermalComparator (THM-02, isolated by the same NTC part's
  1500VAC construction as the heatsink sensor, installation UNVERIFIED),
  SecondaryOCPComparator (OCP-02, not instantiated -- dormant, but its
  own docstring already documents a ~170V common-mode hazard if wired up
  as written), and LogicUVLOComparator (UVL-02, entirely SELV-internal,
  not a crossing).
- Falsifier re-run: gnd/PWR_RTN remain distinct nets (80/17 pins, up from
  74/17 pre-rebase), same 4 deliberate isolation devices straddling both.
- make netlist, make schematics, and kicad-cli sch erc re-run on the
  rebased/regenerated tree; fresh numbers in
  docs/hardware/SELV_ISOLATION_REDESIGN.md (492 ERC warnings / 0 errors,
  same three pre-existing generic categories as before the rebase).

Everything from the original change is preserved: star-join deletion,
PE bond, H11L1 ZCD isolation, the +340V_BUS -> +170V_BUS rename, and the
RTDSensing docstring correction. uvlo_logic.fault.line's deliberate
test-point-only termination (documented elsewhere as intentional) is
left untouched.

Co-Authored-By: Claud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
Parts:
- C10, C13, C16: value GRM188R71E104KA01D -> C0603C104K5RACTU; symbol GRM188R71E104KA01D -> C0603C104K5RACTU
Changed lines of the file:
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@@
   )
   (symbol
-    (lib_id "GRM188R71E104KA01D")
+    (lib_id "C0603C104K5RACTU")
     (at 50.80 50.80 0)
     (unit 1)
@@
     (dnp no)
     (property "Reference" "C10" (at 50.80 48.26 0) (effects (font (size 1.27 1.27))))
-    (property "Value" "GRM188R71E104KA01D" (at 50.80 53.34 0) (effects (font (size 1.27 1.27))))
+    (property "Value" "C0603C104K5RACTU" (at 50.80 53.34 0) (effects (font (size 1.27 1.27))))
     (property "Footprint" "Capacitor_SMD:C_0603_1608Metric" (at 50.80 50.80 0) (effects (font (size 1.27 1.27)) hide))
     (pin "1")
@@
   )
   (symbol
-    (lib_id "GRM188R71E104KA01D")
+    (lib_id "C0603C104K5RACTU")
     (at 170.80 50.80 0)
     (unit 1)
@@
     (dnp no)
     (property "Reference" "C13" (at 170.80 48.26 0) (effects (font (size 1.27 1.27))))
-    (property "Value" "GRM188R71E104KA01D" (at 170.80 53.34 0) (effects (font (size 1.27 1.27))))
+    (property "Value" "C0603C104K5RACTU" (at 170.80 53.34 0) (effects (font (size 1.27 1.27))))
     (property "Footprint" "Capacitor_SMD:C_0603_1608Metric" (at 170.80 50.80 0) (effects (font (size 1.27 1.27)) hide))
     (pin "1")
@@
   )
   (symbol
-    (lib_id "GRM188R71E104KA01D")
+    (lib_id "C0603C104K5RACTU")
     (at 90.80 80.80 0)
     (unit 1)
@@
     (dnp no)
     (property "Reference" "C16" (at 90.80 78.26 0) (effects (font (size 1.27 1.27))))
-    (property "Value" "GRM188R71E104KA01D" (at 90.80 83.34 0) (effects (font (size 1.27 1.27))))
+    (property "Value" "C0603C104K5RACTU" (at 90.80 83.34 0) (effects (font (size 1.27 1.27))))
     (property "Footprint" "Capacitor_SMD:C_0603_1608Metric" (at 90.80 80.80 0) (effects (font (size 1.27 1.27)) hide))
     (pin "1")
