File: pcb/power_management.kicad_sch (KiCad schematic)
At the start: 13 parts, among them U4 LMR51430XDDCR

Commit message: chore(ci): regenerate schematics from netlist after K3 swap (fix 7/7 drift gate)
The K3 RT314012 swap regenerated elec/build/default.net but the 7 KiCad
schematics in pcb/ were never regenerated from it, so the schematic-drift
gate failed all 7 sheets. Run scripts/gen_schematics.py (make schematics)
to re-derive them from the netlist: G5LE-1 -> RT314012 symbol/footprint on
k_dis1/k_dis2 plus netlist UUID churn. Oracle (kicad-cli connectivity
isomorphism) passes: 516 pin assignments, 108 nets.
Parts:
- C11, C12: value GRM32ER71E106KA12L -> GRM32ER71E226KE15L
- C15: value GRM32ER71E106KA12L -> GRM32ER71E107ME15L
- R21: value RC0603FR-0710KL -> RC0603FR-07100KL
- R22: value RC0603FR-0710KL -> RC0603FR-0722K1L
Changed lines of the file:
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@@
     (dnp no)
     (property "Reference" "C11" (at 90.80 48.26 0) (effects (font (size 1.27 1.27))))
-    (property "Value" "GRM32ER71E106KA12L" (at 90.80 53.34 0) (effects (font (size 1.27 1.27))))
+    (property "Value" "GRM32ER71E226KE15L" (at 90.80 53.34 0) (effects (font (size 1.27 1.27))))
     (property "Footprint" "Capacitor_SMD:C_1210_3225Metric" (at 90.80 50.80 0) (effects (font (size 1.27 1.27)) hide))
     (pin "1")
@@
     (dnp no)
     (property "Reference" "C12" (at 130.80 48.26 0) (effects (font (size 1.27 1.27))))
-    (property "Value" "GRM32ER71E106KA12L" (at 130.80 53.34 0) (effects (font (size 1.27 1.27))))
+    (property "Value" "GRM32ER71E226KE15L" (at 130.80 53.34 0) (effects (font (size 1.27 1.27))))
     (property "Footprint" "Capacitor_SMD:C_1210_3225Metric" (at 130.80 50.80 0) (effects (font (size 1.27 1.27)) hide))
     (pin "1")
@@
     (dnp no)
     (property "Reference" "C15" (at 50.80 78.26 0) (effects (font (size 1.27 1.27))))
-    (property "Value" "GRM32ER71E106KA12L" (at 50.80 83.34 0) (effects (font (size 1.27 1.27))))
+    (property "Value" "GRM32ER71E107ME15L" (at 50.80 83.34 0) (effects (font (size 1.27 1.27))))
     (property "Footprint" "Capacitor_SMD:C_1210_3225Metric" (at 50.80 80.80 0) (effects (font (size 1.27 1.27)) hide))
     (pin "1")
@@
     (dnp no)
     (property "Reference" "R21" (at 50.80 108.26 0) (effects (font (size 1.27 1.27))))
-    (property "Value" "RC0603FR-0710KL" (at 50.80 113.34 0) (effects (font (size 1.27 1.27))))
+    (property "Value" "RC0603FR-07100KL" (at 50.80 113.34 0) (effects (font (size 1.27 1.27))))
     (property "Footprint" "Resistor_SMD:R_0603_1608Metric" (at 50.80 110.80 0) (effects (font (size 1.27 1.27)) hide))
     (pin "1")
@@
     (dnp no)
     (property "Reference" "R22" (at 90.80 108.26 0) (effects (font (size 1.27 1.27))))
-    (property "Value" "RC0603FR-0710KL" (at 90.80 113.34 0) (effects (font (size 1.27 1.27))))
+    (property "Value" "RC0603FR-0722K1L" (at 90.80 113.34 0) (effects (font (size 1.27 1.27))))
     (property "Footprint" "Resistor_SMD:R_0603_1608Metric" (at 90.80 110.80 0) (effects (font (size 1.27 1.27)) hide))
     (pin "1")
