File: pcb/temper.kicad_sch (KiCad schematic)
At the start: 0 parts

Commit message: feat(schematics): generate KiCad schematics from atopile netlist (#209)
* feat(identity): collapse board inventory to one quarantined fixture

U1 of plan 2026-07-15-001:
- Delete 14 duplicate/config-capture .kicad_pcb files (all 33-component fixtures)
- Move the one actively-referenced fixture to pcb/benchmarks/temper_fixture_33.kicad_pcb
- Add pcb/benchmarks/README.md documenting the quarantine and sunset
- Repoint golden_manifest.yaml and Makefile (PCB_FILE) at the new fixture location
- The power_pcb_dataset/corpus copy is left in place (self-contained benchmark dataset)

* feat(identity): config-board binding mechanism (U2)

Plan 2026-07-15-001, unit U2:
- config_board_binding.py: extract_config_refs + verify_config_matches_netlist
  fail-closed subset check, refs derived from files, no hand-declared counts.
- 12 synthetic-fixture tests cover: list-keys/single-ref-keys/extraction,
  fixture-refs-rejected-against-production (the exact U_GATE zero-overlap
  case), empty/partial/large-missing, extract-then-verify integration.
- The four existing config files are NOT migrated — all were authored against
  the 33-component fixture with zero overlap with the production netlist.
  They will correctly fail the gate once wired into InputStage (deferred to
  unit U4, Phase B). Production configs are authored/derived after the
  schematic-generation plan delivers the real board.
- Plan doc updated with status note recording this gap explicitly.

* ci: fix hidden-coupling workflow output capture

- Pipe CLI output to .drift-output.txt (was silently reading nonexistent file)
- Surface "could not analyze" pairs when no hidden coupling found (still useful)
- Fix if: condition to fire on always() not tied to exit code

* ci: repoint workflows at quarantined fixture after U1 board move

U1 deleted pcb/temper.kicad_pcb and moved the fixture to
pcb/benchmarks/temper_fixture_33.kicad_pcb. Repoint the 11 hardcoded
references across golden-check, health-digest, metrics-record,
pr-pip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
Other:
- removed sheet User_Interface
- sheet Half_Bridge ports: added +15V, +340V_BUS, +3V3, DC_BUS_RTN, PWM_HS, PWM_LS, SHUTDOWN, gnd; removed DC_BUS+, DC_BUS-, I_SENSE, PWM_H, PWM_L, SHUTDOWN_N, SWITCH_NODE
- sheet MCU ports: added +3V3, PWM_HS, PWM_LS, RTD_CS_N, RTD_SCK, RTD_SDI, RTD_SDO, SHUTDOWN, WDT_RESET_N, gnd, safety-line, safety-line-1, safety-line-2; removed +3.3V, FAULT_STATUS, I2C_SCL, I2C_SDA, PWM_H, PWM_L, RESET_N, RTD_CS, RUNAWAY_CUT, SPI_MISO, SPI_MOSI, SPI_SCK, ZCD
- sheet Power_Input ports: added +340V_BUS, DC_BUS_RTN, gnd; removed AC_L, AC_N, DC_BUS+, DC_BUS-, PE, ZCD
- sheet Power_Management ports: added +3V3, gnd; removed +3.3V, DC_BUS+, PGOOD
- sheet Safety_Interlock ports: added +340V_BUS, +3V3, RTD_HW_FAULT, SHUTDOWN, WDT_RESET_N, gnd, safety-line, safety-line-1, safety-line-2; removed +15V, +3.3V, DC_BUS+, FAULT_STATUS, NTC_SENSE, OCP_FAULT, OVP_FAULT, RESET_N, RUNAWAY_CUT, SHUTDOWN_N, THERMAL_FAULT, WDT_FAULT
- sheet Sensing ports: added +3V3, RTD_CS_N, RTD_HW_FAULT, RTD_SCK, RTD_SDI, RTD_SDO, gnd; removed +15V, +3.3V, I2C_SCL, I2C_SDA, NTC_SENSE, RTD_CS, SPI_MISO, SPI_MOSI, SPI_SCK
- note added: "TEMPER INDUCTION COOKER GENERATED -- do not hand-edit edit elec/src/*.ato and run make schematics 6 Sheets: Power_Input Half_Bridge Power_Management Safety_Interlock (inc. ct_sense) Sensing MCU"
- note removed: "TEMPER INDUCTION COOKER Hierarchical Design Overview Power Flow: AC Mains (120V) → Voltage Doubler → DC Bus (340V) → Half-Bridge → Resonant Tank → Coil Control Flow: ESP32-S3 → PWM → Gate Driver → IGBTs ← ADC ← CT Sensing ← SPI ← Temperature Sensing Safety: OCP + OVP + Thermal + Watchdog → SHUTDOWN_N Power Rails: +3.3V (MCU, Logic) +15V (Gate Driver, Safety Logic) +5V (Isolated Sensors)"

Commit message: chore: regenerate schematics from atopile netlist (#228)
Generated from elec/build/default.net via gen_schematics.py.
Adds 23 new components from discharge (17), aux_supply (4), and
thermal (2) modules that were previously un-mapped and absent.
Root sheet layout re-stacked with dynamic spacing.
Other:
- sheet Half_Bridge ports: added PWR_RTN, tank-out; removed gnd
- sheet MCU ports: added DISCHARGE_CTRL, PWR_RTN, V_BUS_SENSE, ZCD; removed gnd
- sheet Power_Input ports: added DISCHARGE_CTRL, PWR_RTN, ZCD; removed gnd
- sheet Power_Management ports: added +340V_BUS, PWR_RTN; removed gnd
- sheet Safety_Interlock ports: added +15V, PWR_RTN, V_BUS_SENSE, tank-out; removed gnd
- sheet Sensing ports: added PWR_RTN; removed gnd
