File: pcb/temper.kicad_sch (KiCad schematic)
At the start: 0 parts

Commit message: fix: board outline placeholder, ten dead CI gates, and the measurement discipline to catch them (#344)
* fix(router): generalize forced-segment fail-closed gate to every net class

_allow_forced_segments() previously only failed closed for HV/AC-class
nets (R6 of the property-test-hardening plan). Every other net --
including congested power/ground nets like vcc, +3V3, PWR_RTN -- still
fell back to a raw, zero-clearance forced segment when the plain A*
pathfinder couldn't find a legal path, which is why shorting_items
didn't improve after the netclass-clearance wiring fix landed.

The gate now disallows forced segments unconditionally, for every net
class, tree-route context, and design_rules state -- reusing the
existing failed_nets/RoutingFailureReport interception plumbing in
attempt_route(), which was already net-class-agnostic.

Also fixes two pre-existing test gaps discovered along the way:
TestHVACForcedSegmentFailClosed's HV/AC tests used net names
(SW_NODE, AC_L) that are themselves excluded from A* by
_should_route()'s pattern matching, so they never actually exercised
the gate -- new tests use non-excluded names that carry the same
safety classification via design_rules instead. And
test_signal_net_still_allows_forced_segments asserted the exact
opposite of the new uniform behavior; flipped and renamed.

See docs/plans/2026-07-24-001-fix-forced-segment-fail-closed-plan.md
(U1, U2).

* test(router): property-test coverage for uniform forced-segment fail-closed

Sweeps every configured net class (plus unclassified) against grids
guaranteed unroutable by construction, proving no forced segment ever
survives and every such net is honestly reported failed. Fails red
against the pre-generalization gate, passes green after -- confirmed
both ways.

Adds unroutable_wall_grids() to astar_property_strategies.py: unlike
grids()'s Bernoulli obstacle density (which may or may not leave a
path open), this guarantees genuine unroutability via a full-height
wall, needed t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
Other:
- sheet Half_Bridge ports: added +170V_BUS, gnd; removed +340V_BUS, PWR_RTN
- sheet MCU ports: added ZCD_ISO, gnd, safety-line-3; removed PWR_RTN, ZCD, safety-line-1
- sheet Power_Input ports: added +170V_BUS, +3V3, ZCD_ISO, gnd; removed +340V_BUS, ZCD
- sheet Power_Management ports: added +170V_BUS, gnd; removed +340V_BUS
- sheet Safety_Interlock ports: added +170V_BUS, gnd, safety-line-3; removed +340V_BUS, safety-line-1
- sheet Sensing ports: added gnd; removed PWR_RTN
