File: pcb/temper.kicad_sch (KiCad schematic)
At the start: 0 parts

Commit message: chore(ci): regenerate schematics from netlist after K3 swap (fix 7/7 drift gate)
The K3 RT314012 swap regenerated elec/build/default.net but the 7 KiCad
schematics in pcb/ were never regenerated from it, so the schematic-drift
gate failed all 7 sheets. Run scripts/gen_schematics.py (make schematics)
to re-derive them from the netlist: G5LE-1 -> RT314012 symbol/footprint on
k_dis1/k_dis2 plus netlist UUID churn. Oracle (kicad-cli connectivity
isomorphism) passes: 516 pin assignments, 108 nets.
Other:
- sheet Half_Bridge ports: added none; removed +15V
- sheet Safety_Interlock ports: added OVP_VREF_2V5; removed none
- sheet Sensing ports: added OVP_VREF_2V5; removed none
