File: pcb/temper.kicad_sch (KiCad schematic)
At the start: 0 parts

Commit message: fix(pcb): regenerate stale schematic against current elec/src (spike)
pcb/temper.kicad_sch was last regenerated 2026-08-03; elec/src gained the
OCP-02 second-CT module and J_RTD1 pan-probe connector (2026-08-07/08-08)
and lost the ZCD-opto circuit (2026-08-07) without a schematic resync,
leaving scripts/check_erc_off_grid_consequence.py red with 86 MISMATCH
findings on unmodified code.

Diagnosis (docs/evidence/2026-08-11-schematic-elec-drift.md): 81 of the 86
are pure designator-identity churn from the same RENUMBERED cascade
check_netlist_board_reconciliation.py already reports independently (same
physical nets, different (ref,pin) labels); 5 are nets the stale drawing
never had at all (the new OCP-02/pan-probe circuitry). Zero net names that
today's netclass work depends on (ac_l, ac_n, gnd, +170V_BUS, SW_NODE,
GATE_HS/LS, RTD/SPI) were added, removed, or renamed.

Regenerated pcb/*.kicad_sch only (oracle-verified isomorphic to
elec/build/default.net; ERC ratchet still passes at 495<=498 warnings,
0 errors; off-grid-consequence gate 86->1, the residual being a genuine
single-pin net (ac_l) exposed by the ZCD deletion, not a new defect).

The board (pcb/temper.kicad_pcb) is untouched and remains out of sync
with elec/src independently of this fix -- neither caused nor cured by a
schematic regen, since no board-facing gate reads the schematic. 125
reconciliation findings / 13 footprint-drift findings persist unchanged:
6 components (J1, C37, U19, T2, R65, TP3) need board placement and 7
stale ZCD-circuit components (D2, R6-R10, U3) need removal, on a board
currently 0/110 routed. That is a CP-SAT placement decision for the
board owner, not attempted here.

Co-Authored-By: Claude Opus 5 (1M context) <noreply@anthropic.com>
Other:
- sheet Half_Bridge ports: added hb-gnd; removed DC_BUS_RTN
- sheet MCU ports: added none; removed ZCD_ISO
- sheet Power_Input ports: added none; removed +3V3, ZCD_ISO
- sheet Safety_Interlock ports: added DC_BUS_RTN, OCP2_VREF_2V5, hb-gnd; removed OVP_VREF_2V5
- sheet Sensing ports: added OCP2_VREF_2V5; removed OVP_VREF_2V5
