File: pcb/power_input.kicad_sch (KiCad schematic)
At the start: 41 parts, among them K1 G4A-1A-E DC12, K2 G5LE-1 DC12, K3 G5LE-1 DC12, Q1 AO3400A, Q2 AO3400A, U1 MUR1560G, U2 MUR1560G

Commit message: fix(hardware): float SELV control domain, remove star-point ground join
Removes `power_return ~ gnd`, which shorted the AuxSupply IRM-10-15's
4.2kVAC isolation barrier by making the SELV control-domain ground the
same net as the HV doubler midpoint (which tracks AC Neutral). SELV
ground is now bonded directly to protective earth instead, reusing the
existing Y1-cap PE bond point on the HV side without disturbing it.

Isolates the zero-crossing-detect signal with a new H11L1 optocoupler
(verified datasheet pinout/ratings), resolving the project's own
pre-existing TODO. Corrects the "+340V_BUS" net name/comment on
dc_bus_plus, which is actually the +170V half-bus of the Delon doubler
-- that wrong name is what would cause OVP-01's reference divider to be
mistuned by 2x if someone trusted it over the topology; OVPComparator's
docstring now carries the derivation and a warning against that.
Updates RTDSensing's docstring to state what is actually true post-fix
rather than an unqualified isolation claim the netlist didn't fully
support.

Full crossing survey, falsifier result, netlist evidence that gnd and
PWR_RTN are now separate nets, ERC results, and ranked open items
(principally: the OVP-01 bus-sense divider still bridges HV into gnd
resistively and needs a separate part addition to isolate) are in
docs/hardware/SELV_ISOLATION_REDESIGN.md.

Co-Authored-By: Claude Opus 5 <noreply@anthropic.com>
Parts:
- added R10, R9: RC0603FR-0710KL, Resistor_SMD:R_0603_1608Metric, symbol RC0603FR-0710KL
- added U3: H11L1, Package_DIP:DIP-6_W7.62mm, symbol H11L1
- renumbered R9 to R11, R10 to R12, R11 to R13, R12 to R14, R13 to R15, R14 to R16, R15 to R17, R16 to R18, R17 to R19, R18 to R20
Connections:
- net PWR_RTN: now also U3.2; no longer Q1.3, Q2.3, R18.2, R3.2
- net gnd: now reaches C6.2
- net gnd: now also Q1.3, Q2.3, R18.2, R3.2, U3.5
- net +340V_BUS renamed +170V_BUS
- net ZCD renamed zcd
- net zcd: now also R9.1
- new net +3V3: R10.1, U3.6
- new net ZCD_ISO: R10.2, U3.4
- new net a: R9.2, U3.1
- no-connect marks 3 -> 2
Other:
- moved on the sheet: R11, R12, R13, R14, R15, R16, R17, R18, R19, R2, R20, R3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
