File: output/test_debug2/iteration_1.kicad_pcb (KiCad board)
At the start: 4 copper layers, 100 x 150 mm, 33 parts, among them Q1 IKW40N120H3, Q2 IKW40N120H3

Commit message: fix(power): Remove +5V/+3V3/VCC_BOOT from PowerPlaneStage hardcoded list
ROOT CAUSE FOUND: PowerPlaneStage was overriding LayerAssignmentStage decisions.

Problem:
- LayerAssignmentStage correctly set +5V as is_plane=False (PowerTrace class)
- PowerPlaneStage ran AFTER and overwrote is_plane=True (hardcoded TEMPER_PLANE_NETS)
- Sequential router saw is_plane=True and created plane vias instead of traces

Fix:
- Remove +5V, +3V3, VCC_BOOT from TEMPER_PLANE_NETS
- Only +15V remains as power plane (5A, requires plane per IPC-2221)
- Remove corresponding entries from TEMPER_PLANE_LAYERS
- Add comments referencing TemperPowerTopology for strategy

Results:
- +5V now attempts MST/A* routing (correct!) ✓
- +3V3 improved: 18 → 12 unconnected (-6) ✓
- VCC_BOOT improved: 4 → 2 unconnected (-2) ✓
- +5V: 12 → 22 unconnected (+10) ✗ (routing congestion, not logic error)
- Total: 68 → 81 unconnected (+13) (other regressions: USB_D- +20)

Next steps:
- Routing congestion for +5V (90s routing time, many failures)
- Need adaptive A* iteration limits (Task temper-t4si)
- Need via-in-pad for dense areas (Task temper-z3pl)

Task: temper-zy08 (partial progress)
Routing:
- net USB_D-: track 12.5 -> 21.0 mm
- net USB_D+: track 22.5 -> 14.0 mm
