File: pcb/blocks/mcu/mcu_candidate.kicad_sch (KiCad schematic)
At the start: 0 parts

Commit message: fix(mcu): schematic parity and real SW1/SW2 switch footprint
- block_source.build_strict_pin_map: one entry per unique (reference, pin),
  deduping repeated same-number pads and unconnected; a real switch exposes
  pads 1,1,2,2 and the per-physical-pad emission failed the design-bundle
  gate as duplicate_map. The Rust gate is unchanged and still rejects a
  genuine split pad.
- gen_pcb_skeleton.generate_candidate_board: optional values map sets the
  footprint Value from default.csv part identity (was '?').
- gen_schematics: flat strict-candidate layout with unscoped global labels,
  so net names are 'vcc' not '/MCU/vcc' and single-node compiled nets keep
  their pin; production hierarchy is unchanged.
- block_native._electrical_census: collapse repeated same-number pads to one
  electrical identity for the block judge, retaining pads_all for routing.
- apparatus run mcu-20260910-b: real-switch placement and every-physical-pad
  routing; native check 3x = DRC 0 / unconnected 0 / parity 0 / judge pass.
- package pcb/blocks/mcu re-admitted; ASSISTED-PACKAGE.json updated.

The elec/src/components.ato switch-footprint fix is a concurrent working-tree
change treated as fixed input and is intentionally not part of this commit.
Parts:
- added C1: C0603C104K5RACTU, Capacitor_SMD:C_0603_1608Metric, symbol C0603C104K5RACTU
- added C2: GRM21BR71A106KE51L, Capacitor_SMD:C_0805_2012Metric, symbol GRM21BR71A106KE51L
- added C3: GRM188R71A105KA61D, Capacitor_SMD:C_0603_1608Metric, symbol C0603C104K5RACTU
- added R1, R2: RC0603FR-0710KL, Resistor_SMD:R_0603_1608Metric, symbol RC0603FR-0710KL
- added R3, R4: RC0603FR-074K7L, Resistor_SMD:R_0603_1608Metric, symbol RC0603FR-0710KL
- added SW1, SW2: EVQ-P7A01P, Button_Switch_SMD:SW_SPST_EVQP7A, symbol EVQ-P7A01P
- added U1: ESP32-S3-WROOM-1-N8R8, lib:ESP32-S3-WROOM-1, symbol ESP32-S3-WROOM-1-N8R8
Connections:
- new net adc_i_sense_stub: U1.39
- new net adc_ntc_stub: U1.15
- new net adc_v_bus_stub: U1.38
- new net en: C3.1, R1.2, SW1.1, U1.3
- new net gnd: C1.2, C2.2, C3.2, SW1.2, SW2.2, U1.1
- new net gpio18: U1.11
- new net gpio21: U1.23
- new net gpio35: U1.28
- new net gpio36: U1.29
- new net gpio37: U1.30
- new net io0: R2.2, SW2.1, U1.27
- new net io13: U1.21
- new net io40: U1.33
- new net io41: U1.34
- new net io42: U1.35
- new net io45: U1.26
- new net io46: U1.16
- new net io48: U1.25
- new net mcu-line: U1.18
- new net mcu-line-1: U1.17
- new net mcu-line-2: U1.7
- new net mcu-line-3: U1.9
- new net mcu-line-4: U1.24
- new net mcu-line-5: U1.10
- new net mcu-line-6: U1.22
- new net mcu-line-7: U1.6
- new net mcu-line-8: U1.8
- new net miso: U1.20
- new net mosi: U1.19
- new net pwm_h: U1.4
- new net pwm_l: U1.5
- new net rx: U1.36
- new net scl: R4.2, U1.32
- new net sclk: U1.12
- new net sda: R3.2, U1.31
- new net tx: U1.37
- new net usb_dn: U1.13
- new net usb_dp: U1.14
- new net vcc: C1.1, C2.1, R1.1, R2.1, R3.1, R4.1, U1.2
Other:
- removed sheet MCU
- note added: "MCU CANDIDATE GENERATED -- do not hand-edit P1 U2 strict-candidate path: source-derived starting point, no functional copper claims 1 Sheet (flat): MCU"
- note removed: "MCU CANDIDATE GENERATED -- do not hand-edit P1 U2 strict-candidate path: source-derived starting point, no functional copper claims 1 Sheet: MCU"
