File: pcb/prototypes/buck-reva/buck-reva.kicad_pcb (KiCad board)
At the start: 2 copper layers, 50 x 40 mm, 19 parts, among them J1 TerminalBlock_5.08mm_1x02, J2 TerminalBlock_5.08mm_1x02, U3 ?

Commit message: fix(buck-reva): enable schematic-parity DRC and re-freeze
An adversarial review found the freeze cited '0 schematic-parity' while the DRC command never enabled --schematic-parity. Enable the check and fix everything it surfaced: use global labels so net names match the board (+15V not /+15V), sync board footprint Value/Manufacturer/MPN/Datasheet/Description fields from the schematic (assembly/position output no longer reads '?'), and add H1-H4 mounting-hole symbols to the schematic.

KiCad 10.0.6 DRC with --all-track-errors --schematic-parity --severity-all now reports 0 violations / 0 unconnected / 0 schematic-parity; ERC 0. Re-freeze: manifest sha256 3f77b285623adf3fcdc1ccea152fedbf86431f3404f8b9c7b36003c398beebcb. Also record the via-in-pad assembly note and correct the silk/edge-rule wording.
Parts:
- C10, C13: value ? -> 100nF 50V X7R
- C11, C12: value ? -> 22uF 25V X7R
- C9: value ? -> 10uF 50V X7R
- J1: value TerminalBlock_5.08mm_1x02 -> VIN / GND
- J2: value TerminalBlock_5.08mm_1x02 -> 3V3 / GND
- L2: value ? -> 5.6uH
- R16: value ? -> 100k
- R17: value ? -> 22.1k
- U3: value ? -> LMR51430XDDCR
