File: zapote/power-entry/shunt-repair/candidate/section.kicad_sch (KiCad schematic)
At the start: 54 parts, among them U1 GBJ2510-F, U10 C3D20065D, U11 UCC28180D, U12 10mohm, U13 10ohm, U14 10kohm, U15 1kohm, U16 100kohm, U17 91ohm, U18 220ohm, U19 16.2kohm, U2 0031.2510, U20 200kohm, U21 200kohm, U22 200kohm, U23 200kohm, U24 200kohm, U25 13kohm, U26 40.2kohm, U27 1uF, U28 2.7nF, U29 4.7uF, U3 B82726S2163N030, U30 220nF, U31 1nF, U32 680pF, U33 AO3400A, U34 SS14, U35 BAT54H,115, U36 560uF, U37 560uF, U38 560uF, U39 560uF, U4 SL32 10015, U40 470nF, U41 1nF, U42 1714984, U43 61300211121, U44 61300211121, U45 61300211121, U46 AO3400A, U47 AO3400A, U48 100kohm, U49 100kohm, U5 RT33K012, U50 1kohm, U51 100kohm, U52 1714971, U53 150kohm, U54 150kohm, U6 0.22uF, U7 V150LA10AP, U8 760800301, U9 STW65N65DM2

Commit message: feat: finish bounded PFC switching loss experiment
Parts:
- U10: symbol PowerEntryUnit:STW65N65DM2 -> PowerEntryUnit:STW65N65DM2AG
- U9: value STW65N65DM2 -> STW65N65DM2AG; symbol PowerEntryUnit:STW65N65DM2 -> PowerEntryUnit:STW65N65DM2AG
Changed lines of the file:
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@@
   )
   (symbol
-    (lib_id "PowerEntryUnit:STW65N65DM2")
+    (lib_id "PowerEntryUnit:STW65N65DM2AG")
     (at 151.13 50.80 0)
     (unit 1)
@@
   )
   (symbol
-    (lib_id "PowerEntryUnit:STW65N65DM2")
+    (lib_id "PowerEntryUnit:STW65N65DM2AG")
     (at 537.21 477.52 0)
     (unit 1)
@@
     (dnp no)
     (property "Reference" "U9" (at 537.21 474.98 0) (effects (font (size 1.27 1.27))))
-    (property "Value" "STW65N65DM2" (at 537.21 480.06 0) (effects (font (size 1.27 1.27))))
+    (property "Value" "STW65N65DM2AG" (at 537.21 480.06 0) (effects (font (size 1.27 1.27))))
     (property "Footprint" "Package_TO_SOT_THT:TO-247-3_Vertical" (at 537.21 477.52 0) (effects (font (size 1.27 1.27)) hide))
     (pin "1")
