File: zapote/power-entry/active-rectifier/candidate/section.kicad_sch (KiCad schematic)
At the start: 66 parts, among them U1 TEA2209T/1, U10 C3D20065D, U11 UCC28180D, U12 10mohm, U13 10ohm, U14 10kohm, U15 1kohm, U16 100kohm, U17 91ohm, U18 220ohm, U19 16.2kohm, U2 0031.2510, U20 200kohm, U21 200kohm, U22 200kohm, U23 200kohm, U24 200kohm, U25 13kohm, U26 40.2kohm, U27 1uF, U28 2.7nF, U29 4.7uF, U3 B82726S2163N030, U30 220nF, U31 1nF, U32 680pF, U33 AO3400A, U34 SS14, U35 BAT54H,115, U36 560uF, U37 560uF, U38 560uF, U39 560uF, U4 SL32 10015, U40 470nF, U41 1nF, U42 1714984, U43 61300211121, U44 61300211121, U45 61300211121, U46 AO3400A, U47 AO3400A, U48 100kohm, U49 100kohm, U5 RT33K012, U50 1kohm, U51 100kohm, U52 1714971, U53 150kohm, U54 150kohm, U55 IPW60R017C7, U56 IPW60R017C7, U57 IPW60R017C7, U58 IPW60R017C7, U59 220nF, U6 0.22uF, U60 220nF, U61 2.2uF, U62 10ohm, U63 10ohm, U64 10ohm, U65 10ohm, U66 A70QS50-14F, U7 V150LA10AP, U8 760800301, U9 STW65N65DM2AG

Commit message: fix(zapote): bank-side vsense, corrected trunk widths, fresh suite run
U20 divider top moves to hv_plus per CLOSEOUT bank-side intent.
routes.json B.Cu trunk corrected 4.3->3.0 to match suite-03 copper.
Full common suite on final bytes: 3 TEA spacing fails only.
Connections:
- net BOOST_DIODE_POSITIVE: no longer U20.1
- net PFC_BUS_PLUS_390V: now also U20.1
Changed lines of the file:
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@@
     (property "Datasheet" "" (at 313.69 243.84 0) (effects (font (size 1.27 1.27)) hide))
 )
-  (global_label "BOOST_DIODE_POSITIVE"
+  (global_label "PFC_BUS_PLUS_390V"
     (shape bidirectional)
     (at 298.45 243.84 180)
