File: zapote/power-entry/active-rectifier/candidate/section.kicad_pcb (KiCad board)
At the start: 2 copper layers, 310 x 210 mm, 66 parts, among them U1 TEA2209T/1, U10 C3D20065D, U11 UCC28180D, U12 10mohm, U13 10ohm, U14 10kohm, U15 1kohm, U16 100kohm, U17 91ohm, U18 220ohm, U19 16.2kohm, U2 0031.2510, U20 200kohm, U21 200kohm, U22 200kohm, U23 200kohm, U24 200kohm, U25 13kohm, U26 40.2kohm, U27 1uF, U28 2.7nF, U29 4.7uF, U3 B82726S2163N030, U30 220nF, U31 1nF, U32 680pF, U33 AO3400A, U34 SS14, U35 BAT54H,115, U36 560uF, U37 560uF, U38 560uF, U39 560uF, U4 SL32 10015, U40 470nF, U41 1nF, U42 1714984, U43 61300211121, U44 61300211121, U45 61300211121, U46 AO3400A, U47 AO3400A, U48 100kohm, U49 100kohm, U5 RT33K012, U50 1kohm, U51 100kohm, U52 1714971, U53 150kohm, U54 150kohm, U55 IPW60R017C7, U56 IPW60R017C7, U57 IPW60R017C7, U58 IPW60R017C7, U59 220nF, U6 0.22uF, U60 220nF, U61 2.2uF, U62 10ohm, U63 10ohm, U64 10ohm, U65 10ohm, U66 A70QS50-14F, U7 V150LA10AP, U8 760800301, U9 STW65N65DM2AG

Commit message: fix(zapote): validate active rectifier and repair nominal-current routing
Bind the 66-part active source graph, intentional NC pads, half-cycle currents,
fused-bank pulses, domains and loops into the existing Rust unit suite.
Keep passive loss and thermal evidence explicitly inapplicable.

Retain fresh native and common-suite evidence, clear nine route-spacing and
eight nominal branch-current findings, and preserve three TEA package gaps
as failures. Hardware and protection qualification remain incomplete.
Routing:
- net RECTIFIER_L: track 369.0 -> 373.1 mm
- net RECTIFIER_NEGATIVE: track 250.2 -> 252.4 mm
- net BOOST_DIODE_POSITIVE: track 223.9 -> 225.9 mm
- net RECTIFIER_POSITIVE: track 217.8 -> 216.4 mm
Changed lines of the file:
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@@
 	)
 	(segment
-		(start -13.1 118)
-		(end 5 118)
-		(width 3)
+		(start -13.1 116)
+		(end 5 116)
+		(width 4.3)
 		(layer "F.Cu")
 		(net "RECTIFIER_NEGATIVE")
@@
 	)
 	(segment
-		(start 20 123.5)
+		(start 20 120)
 		(end 30 123.5)
-		(width 3)
+		(width 4.3)
 		(layer "F.Cu")
 		(net "RECTIFIER_NEGATIVE")
@@
 	(segment
 		(start -13.1 135)
-		(end -13.1 118)
-		(width 3)
+		(end -13.1 116)
+		(width 4.3)
 		(layer "F.Cu")
 		(net "RECTIFIER_NEGATIVE")
@@
 	)
 	(segment
-		(start 5 118)
-		(end 20 123.5)
-		(width 3)
+		(start 5 116)
+		(end 20 120)
+		(width 4.3)
 		(layer "F.Cu")
 		(net "RECTIFIER_NEGATIVE")
@@
 	)
 	(segment
-		(start 167.9625 125.5)
+		(start 167.9625 127)
 		(end 167.9625 126)
 		(width 0.6)
@@
 	)
 	(via
-		(at 167.9625 125.5)
+		(at 167.9625 127)
 		(size 0.8)
 		(drill 0.4)
@@
 	(segment
 		(start 120.45 122)
-		(end 120.45 125.5)
+		(end 120.45 127)
 		(width 0.6)
 		(layer "B.Cu")
@@
 	)
 	(segment
-		(start 120.45 125.5)
-		(end 167.9625 125.5)
+		(start 120.45 127)
+		(end 167.9625 127)
 		(width 0.6)
 		(layer "B.Cu")
@@
 	)
 	(segment
-		(start 5 130)
+		(start 35.08 131)
 		(end 35.08 130)
-		(width 3)
+		(width 4.3)
 		(layer "F.Cu")
 		(net "RECTIFIER_L")
@@
 		(start -61.55 145)
 		(end -5 145)
-		(width 3)
+		(width 4.3)
 		(layer "F.Cu")
 		(net "RECTIFIER_L")
@@
 	)
 	(segment
+		(start 20 131)
+		(end 35.08 131)
+		(width 4.3)
+		(layer "F.Cu")
+		(net "RECTIFIER_L")
+	)
+	(segment
 		(start -61.55 135)
 		(end -61.55 145)
-		(width 3)
+		(width 4.3)
 		(layer "F.Cu")
 		(net "RECTIFIER_L")
@@
 	(segment
 		(start -5 145)
-		(end 5 130)
-		(width 3)
+		(end 5 127)
+		(width 4.3)
 		(layer "F.Cu")
 		(net "RECTIFIER_L")
@@
 		(end 129 171)
 		(width 6)
+		(layer "F.Cu")
+		(net "RECTIFIER_L")
+	)
+	(segment
+		(start 5 127)
+		(end 20 131)
+		(width 4.3)
 		(layer "F.Cu")
 		(net "RECTIFIER_L")
@@
 	(segment
 		(start -38.525 108.555)
-		(end -37 108.555)
+		(end -38.525 106)
 		(width 0.35)
 		(layer "F.Cu")
@@
 	)
 	(via
-		(at -37 108.555)
+		(at -38.525 106)
 		(size 0.8)
 		(drill 0.4)
@@
 	)
 	(segment
-		(start -37 108.555)
+		(start -38.525 106)
 		(end -37 87)
 		(width 0.5)

Commit message: fix(zapote): bank-side vsense, corrected trunk widths, fresh suite run
U20 divider top moves to hv_plus per CLOSEOUT bank-side intent.
routes.json B.Cu trunk corrected 4.3->3.0 to match suite-03 copper.
Full common suite on final bytes: 3 TEA spacing fails only.
Connections:
- U20 pad 1: BOOST_DIODE_POSITIVE -> PFC_BUS_PLUS_390V
Routing:
- net BOOST_DIODE_POSITIVE: track 225.9 -> 172.4 mm, vias 4 -> 3
- net PFC_BUS_PLUS_390V: track 374.6 -> 414.6 mm

Commit message: feat(zapote): diode-side feedback ECO construction checkpoint
U20.1 now senses BOOST_DIODE_POSITIVE (source-04, strict native bridge,
regenerated schematic, precise KiCad ECO on the clean routed board).
Board a725929a..., schematic b32d6cdb...; exact replay recipe retained in
REPRODUCE.md. Fresh common suite: six units INDETERMINATE, power-entry
FAIL only on the three existing TEA gaps. Native ERC/DRC zero violations.
zapote-erc contract and harness fixtures rebound to the ECO native.json
with a fail-closed mutant for stranding regulation on the bank. Scoped
ECO replay verified independently this session from commit a2536ee14;
full fresh-skeleton replay remains failed/retained (failed-full-replay).
Connections:
- U20 pad 1: PFC_BUS_PLUS_390V -> BOOST_DIODE_POSITIVE
Routing:
- net BOOST_DIODE_POSITIVE: track 172.4 -> 226.1 mm, vias 3 -> 4
- net PFC_BUS_PLUS_390V: track 414.6 -> 374.6 mm
Changed lines of the file:
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@@
 			(layers "F.Cu" "F.Mask" "F.Paste")
 			(roundrect_rratio 0.204082)
-			(net "PFC_BUS_PLUS_390V")
+			(net "BOOST_DIODE_POSITIVE")
 		)
 		(pad "2" smd roundrect
@@
 	)
 	(segment
+		(start 167.9625 126)
+		(end 165 130)
+		(width 0.6)
+		(layer "F.Cu")
+		(net "BOOST_DIODE_POSITIVE")
+	)
+	(segment
 		(start 170.65 22)
 		(end 181.35 22)
@@
 	)
 	(via
+		(at 165 130)
+		(size 1.2)
+		(drill 0.6)
+		(layers "F.Cu" "B.Cu")
+		(net "BOOST_DIODE_POSITIVE")
+	)
+	(via
 		(at 115 90)
 		(size 1.2)
@@
 	)
 	(segment
+		(start 135 115)
+		(end 120 113)
+		(width 0.6)
+		(layer "B.Cu")
+		(net "BOOST_DIODE_POSITIVE")
+	)
+	(segment
 		(start 115 95)
 		(end 115 88)
@@
 	)
 	(segment
+		(start 155 125)
+		(end 145 120)
+		(width 0.6)
+		(layer "B.Cu")
+		(net "BOOST_DIODE_POSITIVE")
+	)
+	(segment
 		(start 120 100)
 		(end 115 95)
@@
 	)
 	(segment
-		(start 120 113)
-		(end 120.45 122)
-		(width 3)
+		(start 165 130)
+		(end 155 125)
+		(width 0.6)
 		(layer "B.Cu")
 		(net "BOOST_DIODE_POSITIVE")
 	)
 	(segment
-		(start 167.9625 121)
-		(end 203 121)
+		(start 145 120)
+		(end 135 115)
 		(width 0.6)
-		(layer "F.Cu")
-		(net "PFC_BUS_PLUS_390V")
+		(layer "B.Cu")
+		(net "BOOST_DIODE_POSITIVE")
+	)
+	(segment
+		(start 120 113)
+		(end 120.45 122)
+		(width 3)
+		(layer "B.Cu")
+		(net "BOOST_DIODE_POSITIVE")
 	)
 	(segment
@@
 		(layer "F.Cu")
 		(net "PFC_BUS_PLUS_390V")
-	)
-	(segment
-		(start 167.9625 126)
-		(end 167.9625 121)
-		(width 0.6)
-		(layer "F.Cu")
-		(net "PFC_BUS_PLUS_390V")
