File: zapote/power-stage-120v/prototype-closure/round5/boards/central/native/ANALOG_GUARD_4.kicad_sch (KiCad schematic)
At the start: 12 parts, among them U9 TLV3201AIDBVR

Commit message: WIP snapshot of worktrees/mit-product-guidance (2026-10-08)
Uncommitted Codex prototype-closure work (round5 boards, round6
investigation, firmware power adapter), snapshotted without touching the
worktree. Raw solver output under output/temper-prototype-closure/ is
not included.

Co-Authored-By: Claude Opus 5.5 (1M context) <noreply@anthropic.com>
Parts:
- R62: value 1.56MR 0.1% TNPW06031M56BEEA -> 1.56MR 0.1% TNPW12061M56BEEA; footprint Resistor_SMD:R_0603_1608Metric -> Resistor_SMD:R_1206_3216Metric
