File: zapote/power-stage-120v/prototype-closure/round5/boards/central/native/COILS_1.kicad_sch (KiCad schematic)
At the start: 12 parts, among them U72 SN74LVC1G08DBVR, U73 SN74LVC1G08DBVR, U74 SN74LVC1G08DBVR, U75 SN74LVC1G08DBVR, U76 SN74LVC1G08DBVR, U77 SN74LVC1G08DBVR

Commit message: WIP snapshot of worktrees/mit-product-guidance (2026-10-08)
Uncommitted Codex prototype-closure work (round5 boards, round6
investigation, firmware power adapter), snapshotted without touching the
worktree. Raw solver output under output/temper-prototype-closure/ is
not included.

Co-Authored-By: Claude Opus 5.5 (1M context) <noreply@anthropic.com>
Connections:
- net ATTEMPT renamed SOURCE_DRIVE_TIMED
