File: zapote/power-stage-120v/prototype-closure/round5/boards/central/native/HARDWARE_10.kicad_sch (KiCad schematic)
At the start: 12 parts, among them U63 SN74LVC1G32DBVR, U64 SN74LVC1G74DCUR, U65 SN74LVC1G08DBVR, U66 SN74LVC1G74DCUR, U67 SN74LVC1G08DBVR, U68 SN74LVC1G08DBVR

Commit message: WIP snapshot of worktrees/mit-product-guidance (2026-10-08)
Uncommitted Codex prototype-closure work (round5 boards, round6
investigation, firmware power adapter), snapshotted without touching the
worktree. Raw solver output under output/temper-prototype-closure/ is
not included.

Co-Authored-By: Claude Opus 5.5 (1M context) <noreply@anthropic.com>
Connections:
- net ATTEMPT: now also U66.6 (CLR_N); no longer U64.1 (CLR_N), U66.1 (CLR_N)
- net MCU_PRECHARGE_DONE: now also U66.1 (CLK); no longer U66.3 (CLK)
- net POD_3V3: no longer U64.2 (D)
- net TOKEN_CLEAR_N: now reaches U64.6 (CLR_N)
- net PROOF_REQUEST: no longer names the net of U64.3 (Q_N)
- net PROOF_STARTED renamed START_TOKEN
- new net START_QUALIFIED: U64.1 (CLK)
- new net TOKEN_ARM_VALID: U64.2 (D)
