File: zapote/power-stage-120v/prototype-closure/round5/boards/central/native/HARDWARE_11.kicad_sch (KiCad schematic)
At the start: 12 parts, among them U69 SN74LVC1G08DBVR, U70 SN74LVC1G08DBVR, U71 SN74LVC1G74DCUR, U82 SN74LVC1G74DCUR, U83 SN74LVC1G04DBVR, U84 SN74LVC1G08DBVR

Commit message: WIP snapshot of worktrees/mit-product-guidance (2026-10-08)
Uncommitted Codex prototype-closure work (round5 boards, round6
investigation, firmware power adapter), snapshotted without touching the
worktree. Raw solver output under output/temper-prototype-closure/ is
not included.

Co-Authored-By: Claude Opus 5.5 (1M context) <noreply@anthropic.com>
Connections:
- net MCU_BYPASS_PROVEN: now also U71.1 (CLK); no longer U71.3 (CLK)
- net PROOF_CAPTURE_VALID: no longer U71.2 (D)
- net FINAL_PROOF_CLEAR_N: now reaches U71.6 (CLR_N)
- net FINAL_PROOF_CLEAR_N: now also U82.6 (CLR_N)
- net ATTEMPT renamed SUP_RUN_OK_LOCAL
- net SUP_RUN_OK_LOCAL: no longer U71.1 (CLR_N)
- net MCU_RUN: no longer names the net of U82.3 (Q_N)
- new net FINAL_PROOF_VALID: U71.2 (D)
