File: zapote/power-stage-120v/prototype-closure/round5/boards/central/native/HARDWARE_13.kicad_sch (KiCad schematic)
At the start: 9 parts, among them U91 SN74LVC1G08DBVR, U92 SN74LVC1G08DBVR, U93 SN74LVC1G08DBVR, U94 SN74LVC1G08DBVR

Commit message: WIP snapshot of worktrees/mit-product-guidance (2026-10-08)
Uncommitted Codex prototype-closure work (round5 boards, round6
investigation, firmware power adapter), snapshotted without touching the
worktree. Raw solver output under output/temper-prototype-closure/ is
not included.

Co-Authored-By: Claude Opus 5.5 (1M context) <noreply@anthropic.com>
Parts:
- added R151: 10kR CRCW060310K0FKEA, Resistor_SMD:R_0603_1608Metric, symbol Supervisor:Part_R151
- added U116: SN74LVC1G04DBVR, Package_TO_SOT_SMD:SOT-23-5, symbol Supervisor:Part_U116
- added U117: SN74LVC1G04DBVR, Package_TO_SOT_SMD:SOT-23-5, symbol Supervisor:Part_U117
Connections:
- net AUX_0V: now also R151.2, U116.3 (GND), U117.3 (GND)
- net CTRL_HEARTBEAT_OK: now also R151.1
- net POD_3V3: now also U116.5 (VCC), U117.5 (VCC)
- net SUP_RUN_OK_LOCAL: no longer U92.4 (Y)
- new net CMD_KPA: U116.2 (A)
- new net CMD_KPB: U117.2 (A)
- new net KPA_CMD_OFF: U116.4 (Y)
- new net KPB_CMD_OFF: U117.4 (Y)
- new net PRE_ISO_RUN_OK: U92.4 (Y)
- no-connect marks 0 -> 2
