File: zapote/power-stage-120v/prototype-closure/round5/boards/central/native/HARDWARE_6.kicad_sch (KiCad schematic)
At the start: 12 parts, among them U44 SN74LVC1G32DBVR, U45 SN74LVC1G32DBVR, U46 SN74LVC1G08DBVR, U47 SN74LVC1G08DBVR, U48 SN74LVC1G08DBVR, U49 SN74LVC1G08DBVR

Commit message: WIP snapshot of worktrees/mit-product-guidance (2026-10-08)
Uncommitted Codex prototype-closure work (round5 boards, round6
investigation, firmware power adapter), snapshotted without touching the
worktree. Raw solver output under output/temper-prototype-closure/ is
not included.

Co-Authored-By: Claude Opus 5.5 (1M context) <noreply@anthropic.com>
Connections:
- net BYPASS_PROVEN renamed SESSION_BUDGET_OK
