File: zapote/power-stage-120v/prototype-closure/round5/boards/central/native/supervisor.kicad_pcb (KiCad board)
At the start: 4 copper layers, 275 x 240 mm, 440 parts, among them J1 1725669 Phoenix MKDS1/2-3.81, J10 B2B-XH-A(LF)(SN), J11 B6B-XH-A(LF)(SN), J12 B2B-XH-A(LF)(SN), J13 B3B-XH-A(LF)(SN), J14 B4B-XH-A(LF)(SN), J15 B4B-XH-A(LF)(SN), J16 B4B-XH-A(LF)(SN), J17 B2B-XH-A(LF)(SN), J18 B6B-XH-A(LF)(SN), J19 B6B-XH-A(LF)(SN), J2 1725669 Phoenix MKDS1/2-3.81, J20 B6B-XH-A(LF)(SN), J21 B6B-XH-A(LF)(SN), J22 B6B-XH-A(LF)(SN), J23 B2B-XH-A(LF)(SN), J24 B2B-XH-A(LF)(SN), J3 1725669 Phoenix MKDS1/2-3.81, J4 B6B-XH-A(LF)(SN), J5 1725669 Phoenix MKDS1/2-3.81, J6 1725669 Phoenix MKDS1/2-3.81, J7 B3B-XH-A(LF)(SN), J8 B8B-XH-A(LF)(SN), J9 B10B-XH-A(LF)(SN), Q1 IRL540NPBF, Q2 IRL540NPBF, Q3 IRL540NPBF, Q4 IRL540NPBF, U1 LD1117S33TR, U10 TLV3201AIDBVR, U100 ISO7710FDR, U101 ISO7710FDR, U102 ISO7710DR, U103 ISO7710FDR, U104 ISO7710FDR, U105 ISO7710FDR, U106 SN74LVC1G04DBVR, U107 ISO7710FDR, U108 STM32G071RBT6, U11 TLV3201AIDBVR, U12 TLV3201AIDBVR, U13 SN74LVC1G08DBVR, U14 TLV3201AIDBVR, U15 TLV3201AIDBVR, U16 SN74LVC1G08DBVR, U17 TLV3201AIDBVR, U18 TLV3201AIDBVR, U19 SN74LVC1G08DBVR, U2 TPS3820-33DBVR, U20 TLV3201AIDBVR, U21 TLV3201AIDBVR, U22 TLV3201AIDBVR, U23 TLV3201AIDBVR, U24 SN74LVC1G08DBVR, U25 SN74LVC1G08DBVR, U26 SN74LVC1G08DBVR, U27 ADS131M08IPBSR, U28 SN74LVC1G08DBVR, U29 SN74LVC1G08DBVR, U3 TPS3825-50DBVR, U30 SN74LVC1G08DBVR, U31 SN74LVC1G08DBVR, U32 SN74LVC1G08DBVR, U33 SN74LVC1G08DBVR, U34 SN74LVC1G08DBVR, U35 SN74LVC1G08DBVR, U36 SN74LVC1G08DBVR, U37 SN74LVC1G08DBVR, U38 SN74LVC1G08DBVR, U39 SN74LVC1G08DBVR, U4 LM4040A25IDBZR, U40 SN74LVC1G08DBVR, U41 SN74LVC1G08DBVR, U42 SN74LVC1G08DBVR, U43 SN74LVC1G04DBVR, U44 SN74LVC1G32DBVR, U45 SN74LVC1G32DBVR, U46 SN74LVC1G08DBVR, U47 SN74LVC1G08DBVR, U48 SN74LVC1G08DBVR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

Commit message: WIP snapshot of worktrees/mit-product-guidance (2026-10-08)
Uncommitted Codex prototype-closure work (round5 boards, round6
investigation, firmware power adapter), snapshotted without touching the
worktree. Raw solver output under output/temper-prototype-closure/ is
not included.

Co-Authored-By: Claude Opus 5.5 (1M context) <noreply@anthropic.com>
Parts:
- added C148: 22uF GRM32ER71E226KE15L 25V X7R, Capacitor_SMD:C_1210_3225Metric, F.Cu at (195.0, 205.0)
- added C149: 22uF GRM32ER71E226KE15L 25V X7R, Capacitor_SMD:C_1210_3225Metric, F.Cu at (201.0, 205.0)
- added C150: 22uF GRM32ER71E226KE15L 25V X7R, Capacitor_SMD:C_1210_3225Metric, F.Cu at (177.0, 212.0)
- added C151: 22uF GRM32ER71E226KE15L 25V X7R, Capacitor_SMD:C_1210_3225Metric, F.Cu at (177.0, 218.0)
- added C152: 22uF GRM32ER71E226KE15L 25V X7R, Capacitor_SMD:C_1210_3225Metric, F.Cu at (183.0, 218.0)
- added C153: 1uF C1206C105K5RAC 50V, Capacitor_SMD:C_1206_3216Metric, F.Cu at (195.0, 212.0)
- added C154: 1nF C0603C102J5GACTU 50V, Capacitor_SMD:C_0603_1608Metric, F.Cu at (42.0, 221.0)
- added C155: 100nF C0603C104K5RACAUTO, Capacitor_SMD:C_0603_1608Metric, F.Cu at (33.0, 202.0)
- added C156: 1nF C0603C102J5GACTU 50V, Capacitor_SMD:C_0603_1608Metric, F.Cu at (67.0, 221.0)
- added C157: 100nF C0603C104K5RACAUTO, Capacitor_SMD:C_0603_1608Metric, F.Cu at (54.0, 205.0)
- added C158: 1nF C0603C102J5GACTU 50V, Capacitor_SMD:C_0603_1608Metric, F.Cu at (92.0, 221.0)
- added C159: 100nF C0603C104K5RACAUTO, Capacitor_SMD:C_0603_1608Metric, F.Cu at (79.0, 205.0)
- added C160: 1nF C0603C102J5GACTU 50V, Capacitor_SMD:C_0603_1608Metric, F.Cu at (117.0, 221.0)
- added C161: 100nF C0603C104K5RACAUTO, Capacitor_SMD:C_0603_1608Metric, F.Cu at (104.0, 205.0)
- added C162: 1nF C0603C102J5GACTU 50V, Capacitor_SMD:C_0603_1608Metric, F.Cu at (142.0, 221.0)
- added C163: 100nF C0603C104K5RACAUTO, Capacitor_SMD:C_0603_1608Metric, F.Cu at (129.0, 205.0)
- added C164: 100nF C0603C104J5RACTU 50V, Capacitor_SMD:C_0603_1608Metric, F.Cu at (162.0, 222.0)
- added C165: 100nF C0603C104K5RACAUTO, Capacitor_SMD:C_0603_1608Metric, F.Cu at (25.0, 182.0)
- added C166: 100nF C0603C104K5RACAUTO, Capacitor_SMD:C_0603_1608Metric, F.Cu at (35.0, 182.0)
- added C167: 100nF C0603C104K5RACAUTO, Capacitor_SMD:C_0603_1608Metric, F.Cu at (45.0, 182.0)
- added C168: 100nF C0603C104K5RACAUTO, Capacitor_SMD:C_0603_1608Metric, F.Cu at (55.0, 182.0)
- added C169: 100nF C0603C104K5RACAUTO, Capacitor_SMD:C_0603_1608Metric, F.Cu at (65.0, 182.0)
- added C170: 100nF C0603C104K5RACAUTO, Capacitor_SMD:C_0603_1608Metric, F.Cu at (75.0, 182.0)
- added C171: 100nF C0603C104K5RACAUTO, Capacitor_SMD:C_0603_1608Metric, F.Cu at (85.0, 182.0)
- added C172: 100nF C0603C104K5RACAUTO, Capacitor_SMD:C_0603_1608Metric, F.Cu at (95.0, 182.0)
- added C173: 100nF C0603C104K5RACAUTO, Capacitor_SMD:C_0603_1608Metric, F.Cu at (105.0, 182.0)
- added C174: 100nF C0603C104K5RACAUTO, Capacitor_SMD:C_0603_1608Metric, F.Cu at (115.0, 182.0)
- added C175: 100nF C0603C104K5RACAUTO, Capacitor_SMD:C_0603_1608Metric, B.Cu at (24.0, 129.0)
- added C176: 100nF C0603C104K5RACAUTO, Capacitor_SMD:C_0603_1608Metric, F.Cu at (125.0, 182.0)
- added C177: 100nF C0603C104K5RACAUTO, Capacitor_SMD:C_0603_1608Metric, F.Cu at (139.0, 180.0)
- added C178: 100nF C0603C104K5RACAUTO, Capacitor_SMD:C_0603_1608Metric, B.Cu at (32.0, 140.0)
- added C179: 100nF C0603C104K5RACAUTO, Capacitor_SMD:C_0603_1608Metric, B.Cu at (44.0, 140.0)
- added C180: 100nF C0603C104K5RACAUTO, Capacitor_SMD:C_0603_1608Metric, B.Cu at (56.0, 140.0)
- added C181: 100nF C0603C104K5RACAUTO, Capacitor_SMD:C_0603_1608Metric, B.Cu at (68.0, 140.0)
- added C182: 100nF C0603C104K5RACAUTO, Capacitor_SMD:C_0603_1608Metric, B.Cu at (80.0, 140.0)
- added C183: 100nF C0603C104K5RACAUTO, Capacitor_SMD:C_0603_1608Metric, B.Cu at (92.0, 140.0)
- added C184: 100nF C0603C104K5RACAUTO, Capacitor_SMD:C_0603_1608Metric, B.Cu at (104.0, 140.0)
- added C185: 100nF C0603C104K5RACAUTO, Capacitor_SMD:C_0603_1608Metric, B.Cu at (116.0, 140.0)
- added C186: 100nF C0603C104K5RACAUTO, Capacitor_SMD:C_0603_1608Metric, B.Cu at (128.0, 140.0)
- added C187: 100nF C0603C104K5RACAUTO, Capacitor_SMD:C_0603_1608Metric, B.Cu at (140.0, 140.0)
- added C188: 100nF C0603C104K5RACAUTO, Capacitor_SMD:C_0603_1608Metric, B.Cu at (152.0, 140.0)
- added C189: 100nF C0603C104K5RACAUTO, Capacitor_SMD:C_0603_1608Metric, B.Cu at (20.0, 152.0)
- added C190: 100nF C0603C104K5RACAUTO, Capacitor_SMD:C_0603_1608Metric, B.Cu at (32.0, 152.0)
- added C191: 100nF C0603C104K5RACAUTO, Capacitor_SMD:C_0603_1608Metric, B.Cu at (44.0, 152.0)
- added C192: 100nF C0603C104K5RACAUTO, Capacitor_SMD:C_0603_1608Metric, B.Cu at (56.0, 152.0)
- added C193: 100nF C0603C104K5RACAUTO, Capacitor_SMD:C_0603_1608Metric, B.Cu at (68.0, 152.0)
- added C194: 100nF C0603C104K5RACAUTO, Capacitor_SMD:C_0603_1608Metric, B.Cu at (85.0, 153.5)
- added C195: 100nF C0603C104K5RACAUTO, Capacitor_SMD:C_0603_1608Metric, B.Cu at (92.0, 152.0)
- added C196: 100nF C0603C104K5RACAUTO, Capacitor_SMD:C_0603_1608Metric, B.Cu at (107.0, 153.0)
- added C197: 100nF C0603C104K5RACAUTO, Capacitor_SMD:C_0603_1608Metric, B.Cu at (116.0, 153.5)
- added C198: 100nF C0603C104K5RACAUTO, Capacitor_SMD:C_0603_1608Metric, B.Cu at (128.0, 152.0)
- added C199: 100nF C0603C104K5RACAUTO, Capacitor_SMD:C_0603_1608Metric, B.Cu at (140.0, 152.0)
- added C200: 100nF C0603C104K5RACAUTO, Capacitor_SMD:C_0603_1608Metric, B.Cu at (152.0, 152.0)
- added C201: 100nF C0603C104K5RACAUTO, Capacitor_SMD:C_0603_1608Metric, B.Cu at (20.0, 164.0)
- added C202: 100nF C0603C104K5RACAUTO, Capacitor_SMD:C_0603_1608Metric, F.Cu at (26.0, 188.0)
- added C203: 100nF C0603C104K5RACAUTO, Capacitor_SMD:C_0603_1608Metric, B.Cu at (32.0, 164.0)
- added C204: 100nF C0603C104K5RACAUTO, Capacitor_SMD:C_0603_1608Metric, B.Cu at (44.0, 165.5)
- added C205: 100nF C0603C104K5RACAUTO, Capacitor_SMD:C_0603_1608Metric, B.Cu at (56.0, 164.0)
- added C206: 100nF C0603C104K5RACAUTO, Capacitor_SMD:C_0603_1608Metric, B.Cu at (68.0, 164.0)
- added C207: 100nF C0603C104K5RACAUTO, Capacitor_SMD:C_0603_1608Metric, B.Cu at (80.0, 164.0)
- added C208: 100nF C0603C104K5RACAUTO, Capacitor_SMD:C_0603_1608Metric, B.Cu at (92.0, 164.0)
- added C209: 100nF C0603C104K5RACAUTO, Capacitor_SMD:C_0603_1608Metric, B.Cu at (104.0, 165.5)
- added C210: 100nF C0603C104K5RACAUTO, Capacitor_SMD:C_0603_1608Metric, B.Cu at (116.0, 164.0)
- added C211: 100nF C0603C104K5RACAUTO, Capacitor_SMD:C_0603_1608Metric, B.Cu at (128.0, 164.0)
- added C212: 100nF C0603C104K5RACAUTO, Capacitor_SMD:C_0603_1608Metric, B.Cu at (164.0, 164.0)
- added C213: 100nF C0603C104K5RACAUTO, Capacitor_SMD:C_0603_1608Metric, B.Cu at (50.0, 80.0)
- added J25: B4B-XH-A(LF)(SN), Connector_JST:JST_XH_B4B-XH-A_1x04_P2.50mm_Vertical, F.Cu at (5.00, 208.0)
- added J26: B4B-XH-A(LF)(SN), Connector_JST:JST_XH_B4B-XH-A_1x04_P2.50mm_Vertical, F.Cu at (8.00, 224.0)
- added N1: PCB copper star 2mm, NetTie:NetTie-2_SMD_Pad2.0mm, F.Cu at (237.0, 228.0)
- added Q5: IRL540NPBF, Package_TO_SOT_THT:TO-220-3_Vertical, F.Cu at (22.0, 207.0)
- added Q6: IRL540NPBF, Package_TO_SOT_THT:TO-220-3_Vertical, F.Cu at (22.0, 220.0)
- added R151: 10kR CRCW060310K0FKEA, Resistor_SMD:R_0603_1608Metric, B.Cu at (117.0, 62.0)
- added R152: 33R CRCW060333R0FKEA, Resistor_SMD:R_0603_1608Metric, B.Cu at (182.0, 166.0)
- added R153: 300R 0.1% TNPW1206300RBEEA, Resistor_SMD:R_1206_3216Metric, F.Cu at (178.0, 205.0)
- added R154: 4.7kR CRCW20104K70FKEF 0.75W, Resistor_SMD:R_2010_5025Metric, F.Cu at (47.0, 215.0)
- added R155: 100kR CRCW0603100KFKEA, Resistor_SMD:R_0603_1608Metric, F.Cu at (35.0, 221.0)
- added R156: 4.7kR CRCW20104K70FKEF 0.75W, Resistor_SMD:R_2010_5025Metric, F.Cu at (72.0, 215.0)
- added R157: 100kR CRCW0603100KFKEA, Resistor_SMD:R_0603_1608Metric, F.Cu at (60.0, 221.0)
- added R158: 4.7kR CRCW20104K70FKEF 0.75W, Resistor_SMD:R_2010_5025Metric, F.Cu at (97.0, 215.0)
- added R159: 100kR CRCW0603100KFKEA, Resistor_SMD:R_0603_1608Metric, F.Cu at (85.0, 221.0)
- added R160: 100kR CRCW0603100KFKEA, Resistor_SMD:R_0603_1608Metric, F.Cu at (104.0, 217.0)
- added R161: 562R CRCW0603562RFKEA, Resistor_SMD:R_0603_1608Metric, F.Cu at (117.0, 208.0)
- added R162: 4.7kR CRCW20104K70FKEF 0.75W, Resistor_SMD:R_2010_5025Metric, F.Cu at (122.0, 215.0)
- added R163: 100kR CRCW0603100KFKEA, Resistor_SMD:R_0603_1608Metric, F.Cu at (110.0, 221.0)
- added R164: 100kR CRCW0603100KFKEA, Resistor_SMD:R_0603_1608Metric, F.Cu at (129.0, 217.0)
- added R165: 562R CRCW0603562RFKEA, Resistor_SMD:R_0603_1608Metric, F.Cu at (142.0, 208.0)
- added R166: 4.7kR CRCW20104K70FKEF 0.75W, Resistor_SMD:R_2010_5025Metric, F.Cu at (147.0, 215.0)
- added R167: 100kR CRCW0603100KFKEA, Resistor_SMD:R_0603_1608Metric, F.Cu at (135.0, 221.0)
- added R168: 10kR CRCW060310K0FKEA, Resistor_SMD:R_0603_1608Metric, F.Cu at (30.0, 185.0)
- added R169: 10kR CRCW060310K0FKEA, Resistor_SMD:R_0603_1608Metric, F.Cu at (35.0, 186.0)
- added R170: 620kR 0.1% TNPW0805620KBEEA, Resistor_SMD:R_0805_2012Metric, F.Cu at (105.0, 187.0)
- added R171: 10kR 0.1% TNPW060310K0BEEA, Resistor_SMD:R_0603_1608Metric, F.Cu at (115.0, 187.0)
- added R172: 10kR 0.1% TNPW060310K0BEEA, Resistor_SMD:R_0603_1608Metric, F.Cu at (125.0, 187.0)
- added R173: 620kR 0.1% TNPW0805620KBEEA, Resistor_SMD:R_0805_2012Metric, F.Cu at (135.0, 187.0)
- added R174: 1kR CRCW06031K00FKEA, Resistor_SMD:R_0603_1608Metric, F.Cu at (28.0, 200.0)
- added R175: 22kR CRCW060322K0FKEA, Resistor_SMD:R_0603_1608Metric, F.Cu at (28.0, 212.0)
- added R176: 1kR CRCW06031K00FKEA, Resistor_SMD:R_0603_1608Metric, F.Cu at (28.0, 214.0)
- added R177: 22kR CRCW060322K0FKEA, Resistor_SMD:R_0603_1608Metric, F.Cu at (28.0, 224.0)
- added R178: 10kR CRCW060310K0FKEA, Resistor_SMD:R_0603_1608Metric, F.Cu at (182.0, 179.0)
- added R179: 39R 1% PR03000203909FAC00 3W, Resistor_THT:R_Axial_DIN0617_L17.0mm_D6.0mm_P25.40mm_Horizontal, F.Cu at (244.0, 180.0)
- added R180: 10kR CRCW060310K0FKEA, Resistor_SMD:R_0603_1608Metric, F.Cu at (267.0, 87.0)
- added R181: 10kR CRCW060310K0FKEA, Resistor_SMD:R_0603_1608Metric, F.Cu at (267.0, 83.0)
- added R182: 10kR CRCW060310K0FKEA, Resistor_SMD:R_0603_1608Metric, F.Cu at (13.0, 186.0)
- added R183: 10kR CRCW060310K0FKEA, Resistor_SMD:R_0603_1608Metric, F.Cu at (13.0, 189.0)
- added U109: TPS7A4700RGWR, Package_DFN_QFN:Texas_RGW0020A_VQFN-20-1EP_5x5mm_P0.65mm_EP3.15x3.15mm, F.Cu at (185.0, 210.0)
- added U110: ISO1211DR, Package_SO:SOIC-8_3.9x4.9mm_P1.27mm, F.Cu at (35.0, 211.0)
- added U111: ISO1211DR, Package_SO:SOIC-8_3.9x4.9mm_P1.27mm, F.Cu at (60.0, 211.0)
- added U112: ISO1211DR, Package_SO:SOIC-8_3.9x4.9mm_P1.27mm, F.Cu at (85.0, 211.0)
- added U113: ISO1211DR, Package_SO:SOIC-8_3.9x4.9mm_P1.27mm, F.Cu at (110.0, 211.0)
- added U114: ISO1211DR, Package_SO:SOIC-8_3.9x4.9mm_P1.27mm, F.Cu at (135.0, 211.0)
- added U115: TPL7407LDR, Package_SO:SOIC-16_3.9x9.9mm_P1.27mm, F.Cu at (155.0, 217.0)
- added U116: SN74LVC1G04DBVR, Package_TO_SOT_SMD:SOT-23-5, F.Cu at (25.0, 177.0)
- added U117: SN74LVC1G04DBVR, Package_TO_SOT_SMD:SOT-23-5, F.Cu at (35.0, 177.0)
- added U118: SN74LVC1G08DBVR, Package_TO_SOT_SMD:SOT-23-5, F.Cu at (45.0, 177.0)
- added U119: SN74LVC1G08DBVR, Package_TO_SOT_SMD:SOT-23-5, F.Cu at (55.0, 177.0)
- added U120: SN74LVC1G08DBVR, Package_TO_SOT_SMD:SOT-23-5, F.Cu at (65.0, 177.0)
- added U121: SN74LVC1G08DBVR, Package_TO_SOT_SMD:SOT-23-5, F.Cu at (75.0, 177.0)
- added U122: SN74LVC1G08DBVR, Package_TO_SOT_SMD:SOT-23-5, F.Cu at (85.0, 177.0)
- added U123: SN74LVC1G08DBVR, Package_TO_SOT_SMD:SOT-23-5, F.Cu at (95.0, 177.0)
- added U124: TLV3201AIDBVR, Package_TO_SOT_SMD:SOT-23-5, F.Cu at (105.0, 177.0)
- added U125: TLV3201AIDBVR, Package_TO_SOT_SMD:SOT-23-5, F.Cu at (115.0, 177.0)
- added U126: SN74LVC1G08DBVR, Package_TO_SOT_SMD:SOT-23-5, B.Cu at (24.0, 132.0)
- added U127: TLV3201AIDBVR, Package_TO_SOT_SMD:SOT-23-5, F.Cu at (125.0, 177.0)
- added U128: TLV3201AIDBVR, Package_TO_SOT_SMD:SOT-23-5, F.Cu at (135.0, 177.0)
- added U129: SN74LVC1G08DBVR, Package_TO_SOT_SMD:SOT-23-5, B.Cu at (32.0, 133.0)
- added U130: SN74LVC1G04DBVR, Package_TO_SOT_SMD:SOT-23-5, B.Cu at (44.0, 135.0)
- added U131: SN74LVC1G04DBVR, Package_TO_SOT_SMD:SOT-23-5, B.Cu at (56.0, 135.0)
- added U132: SN74LVC1G04DBVR, Package_TO_SOT_SMD:SOT-23-5, B.Cu at (68.0, 135.0)
- added U133: SN74LVC1G08DBVR, Package_TO_SOT_SMD:SOT-23-5, B.Cu at (80.0, 135.0)
- added U134: SN74LVC1G08DBVR, Package_TO_SOT_SMD:SOT-23-5, B.Cu at (92.0, 135.0)
- added U135: SN74LVC1G08DBVR, Package_TO_SOT_SMD:SOT-23-5, B.Cu at (104.0, 135.0)
- added U136: SN74LVC1G08DBVR, Package_TO_SOT_SMD:SOT-23-5, B.Cu at (116.0, 135.0)
- added U137: SN74LVC1G08DBVR, Package_TO_SOT_SMD:SOT-23-5, B.Cu at (128.0, 135.0)
- added U138: SN74LVC1G08DBVR, Package_TO_SOT_SMD:SOT-23-5, B.Cu at (140.0, 135.0)
- added U139: SN74LVC1G08DBVR, Package_TO_SOT_SMD:SOT-23-5, B.Cu at (152.0, 135.0)
- added U140: SN74LVC1G08DBVR, Package_TO_SOT_SMD:SOT-23-5, B.Cu at (20.0, 147.0)
- added U141: SN74LVC1G08DBVR, Package_TO_SOT_SMD:SOT-23-5, B.Cu at (32.0, 147.0)
- added U142: SN74LVC1G08DBVR, Package_TO_SOT_SMD:SOT-23-5, B.Cu at (44.0, 147.0)
- added U143: SN74LVC1G08DBVR, Package_TO_SOT_SMD:SOT-23-5, B.Cu at (56.0, 147.0)
- added U144: SN74LVC1G08DBVR, Package_TO_SOT_SMD:SOT-23-5, B.Cu at (68.0, 147.0)
- added U145: SN74LVC1G04DBVR, Package_TO_SOT_SMD:SOT-23-5, B.Cu at (80.0, 147.0)
- added U146: SN74LVC1G08DBVR, Package_TO_SOT_SMD:SOT-23-5, B.Cu at (92.0, 147.0)
- added U147: SN74LVC1G08DBVR, Package_TO_SOT_SMD:SOT-23-5, B.Cu at (104.0, 147.0)
- added U148: SN74LVC1G32DBVR, Package_TO_SOT_SMD:SOT-23-5, B.Cu at (116.0, 147.0)
- added U149: SN74LVC1G08DBVR, Package_TO_SOT_SMD:SOT-23-5, B.Cu at (128.0, 147.0)
- added U150: SN74LVC1G08DBVR, Package_TO_SOT_SMD:SOT-23-5, B.Cu at (140.0, 147.0)
- added U151: SN74LVC1G08DBVR, Package_TO_SOT_SMD:SOT-23-5, B.Cu at (152.0, 147.0)
- added U152: SN74LVC1G08DBVR, Package_TO_SOT_SMD:SOT-23-5, B.Cu at (20.0, 159.0)
- added U153: SN74AHCT125PWR, Package_SO:TSSOP-14_4.4x5mm_P0.65mm, F.Cu at (20.0, 188.0)
- added U154: SN74LVC1G04DBVR, Package_TO_SOT_SMD:SOT-23-5, B.Cu at (32.0, 159.0)
- added U155: SN74LVC1G08DBVR, Package_TO_SOT_SMD:SOT-23-5, B.Cu at (44.0, 159.0)
- added U156: SN74LVC1G08DBVR, Package_TO_SOT_SMD:SOT-23-5, B.Cu at (56.0, 159.0)
- added U157: SN74LVC1G04DBVR, Package_TO_SOT_SMD:SOT-23-5, B.Cu at (68.0, 159.0)
- added U158: SN74LVC1G08DBVR, Package_TO_SOT_SMD:SOT-23-5, B.Cu at (80.0, 159.0)
- added U159: SN74LVC1G08DBVR, Package_TO_SOT_SMD:SOT-23-5, B.Cu at (92.0, 159.0)
- added U160: SN74LVC1G32DBVR, Package_TO_SOT_SMD:SOT-23-5, B.Cu at (104.0, 159.0)
- added U161: SN74LVC1G08DBVR, Package_TO_SOT_SMD:SOT-23-5, B.Cu at (116.0, 159.0)
- added U162: SN74LVC1G08DBVR, Package_TO_SOT_SMD:SOT-23-5, B.Cu at (128.0, 157.5)
- added U163: SN74LVC1G08DBVR, Package_TO_SOT_SMD:SOT-23-5, B.Cu at (164.0, 159.0)
- added U164: SN74LVC1G08DBVR, Package_TO_SOT_SMD:SOT-23-5, B.Cu at (50.0, 75.0)
- C3: value 1uF 12063C105KAT2A -> 1uF C1206C105K5RAC 50V
- R1: value 470R 0.1% TNPW1206470RBEEA -> 82R 1% CRCW251282R0FKEG 1W; footprint Resistor_SMD:R_1206_3216Metric -> Resistor_SMD:R_2512_6332Metric
- R105, R108, R111: value 1MR 0.1% TNPW06031M00BEEA -> 1MR 0.1% TNPW08051M00BEEA; footprint Resistor_SMD:R_0603_1608Metric -> Resistor_SMD:R_0805_2012Metric
- R106, R109: value 681kR 0.1% TNPW0603681KBEEA -> 681kR 0.1% TNPW0805681KBEEA; footprint Resistor_SMD:R_0603_1608Metric -> Resistor_SMD:R_0805_2012Metric
- R110: value 140kR 0.1% TNPW0603140KBEEA -> 191kR 0.1% TNPW0603191KBEEA
- R112: value 523kR 0.1% TNPW0603523KBEEA -> 523kR 0.1% TNPW0805523KBEEA; footprint Resistor_SMD:R_0603_1608Metric -> Resistor_SMD:R_0805_2012Metric
- R130, R132, R134: value 10kR CRCW060310K0FKEA -> 100kR CRCW0603100KFKEA
- R131, R133, R135: value 1kR CRCW06031K00FKEA -> 562R CRCW0603562RFKEA
- R62: value 1.56MR 0.1% TNPW06031M56BEEA -> 1.56MR 0.1% TNPW12061M56BEEA; footprint Resistor_SMD:R_0603_1608Metric -> Resistor_SMD:R_1206_3216Metric
- U1: value LD1117S33TR -> R-78B5.0-1.0; footprint Package_TO_SOT_SMD:SOT-223-3_TabPin2 -> Converter_DCDC:Converter_DCDC_RECOM_R-78HB-0.5_THT
- moved R130 221.9 mm to (32.0, 217.0)
- moved R132 221.9 mm to (54.0, 217.0)
- moved R134 219.4 mm to (79.0, 217.0)
- moved R131 218.0 mm to (42.0, 208.0)
- moved R133 215.4 mm to (67.0, 208.0)
- moved R135 163.4 mm to (92.0, 208.0)
- moved R1 132.3 mm to (256.0, 209.0)
- moved C3 74.7 mm to (158.0, 205.0), turned to 180 degrees
- moved U1 69.2 mm to (165.0, 205.0)
- moved C4 57.8 mm to (174.0, 199.0)
Connections:
- C3 pad 1: POD_5V -> AUX_24V
- J14 pad 3: K1_FB_EXC -> AUX_24V
- J14 pad 4: K1_MIRROR_RAW -> K1_MIRROR_24V
- J15 pad 3: K2_FB_EXC -> AUX_24V
- J15 pad 4: K2_MIRROR_RAW -> K2_MIRROR_24V
- J16 pad 3: KB_FB_EXC -> AUX_24V
- J16 pad 4: KB_MIRROR_RAW -> KB_MIRROR_24V
- Q1 pad 3: AUX_0V -> COIL_RET
- Q2 pad 3: AUX_0V -> COIL_RET
- Q3 pad 3: AUX_0V -> COIL_RET
- Q4 pad 3: AUX_0V -> COIL_RET
- R123 pad 2: AUX_0V -> COIL_RET
- R125 pad 2: AUX_0V -> COIL_RET
- R127 pad 2: AUX_0V -> COIL_RET
- R129 pad 2: AUX_0V -> COIL_RET
- R130 pad 1: K1_MIRROR_RAW -> K1_MIRROR
- R131 pad 1: K1_MIRROR_RAW -> K1_MIRROR_24V
- R131 pad 2: K1_MIRROR -> K1_FB_IN
- R132 pad 1: K2_MIRROR_RAW -> K2_MIRROR
- R133 pad 1: K2_MIRROR_RAW -> K2_MIRROR_24V
- R133 pad 2: K2_MIRROR -> K2_FB_IN
- R134 pad 1: KB_MIRROR_RAW -> KB_MIRROR
- R135 pad 1: KB_MIRROR_RAW -> KB_MIRROR_24V
- R135 pad 2: KB_MIRROR -> KB_FB_IN
- U1 pad 1: AUX_0V -> AUX_24V
- U1 pad 2: POD_3V3 -> AUX_0V
- U1 pad 3: POD_5V -> REG3_5V
- U108 pad 3: unconnected-(U108-PC13-Pad3) -> KPA_MIRROR
- U108 pad 36: ADC_CLKIN -> ADC_MCO_SOURCE
- U108 pad 4: unconnected-(U108-PC14-Pad4) -> KPB_MIRROR
- U108 pad 40: unconnected-(U108-PD8-Pad40) -> CMD_KPA
- U108 pad 41: unconnected-(U108-PD9-Pad41) -> CMD_KPB
- U108 pad 44: unconnected-(U108-PA12-Pad44) -> KPA_FB_EXC
- U108 pad 47: unconnected-(U108-PA15-Pad47) -> KPB_FB_EXC
- U108 pad 5: unconnected-(U108-PC15-Pad5) -> ADMIT
- U44 pad 2: BYPASS_PROVEN -> SESSION_BUDGET_OK
- U51 pad 1: FAULT_CLEAR_N -> RESET_QUALIFIED
- U51 pad 3: RESET_QUALIFIED -> unconnected-(U51-Q_N-Pad3)
- U51 pad 6: unconnected-(U51-Q_N-Pad6) -> FAULT_CLEAR_N
- U57 pad 1: ATTEMPT_CLEAR_N -> ADMIT
- U57 pad 2: POD_3V3 -> ATTEMPT_D
- U57 pad 3: START_QUALIFIED -> unconnected-(U57-Q_N-Pad3)
- U57 pad 6: unconnected-(U57-Q_N-Pad6) -> ATTEMPT_CLEAR_N
- U60 pad 1: PROOF_STARTED -> PROOF_REQUEST
- U64 pad 1: ATTEMPT -> START_QUALIFIED
- U64 pad 2: POD_3V3 -> TOKEN_ARM_VALID
- U64 pad 3: PROOF_REQUEST -> unconnected-(U64-Q_N-Pad3)
- U64 pad 5: PROOF_STARTED -> START_TOKEN
- U64 pad 6: unconnected-(U64-Q_N-Pad6) -> TOKEN_CLEAR_N
- U66 pad 1: ATTEMPT -> MCU_PRECHARGE_DONE
- U66 pad 3: MCU_PRECHARGE_DONE -> unconnected-(U66-Q_N-Pad3)
- U66 pad 6: unconnected-(U66-Q_N-Pad6) -> ATTEMPT
- U71 pad 1: ATTEMPT -> MCU_BYPASS_PROVEN
- U71 pad 2: PROOF_CAPTURE_VALID -> FINAL_PROOF_VALID
- U71 pad 3: MCU_BYPASS_PROVEN -> unconnected-(U71-Q_N-Pad3)
- U71 pad 6: unconnected-(U71-Q_N-Pad6) -> FINAL_PROOF_CLEAR_N
- U72 pad 1: ATTEMPT -> SOURCE_DRIVE_TIMED
- U74 pad 1: ATTEMPT -> SOURCE_DRIVE_TIMED
- U82 pad 1: ATTEMPT -> SUP_RUN_OK_LOCAL
- U82 pad 3: MCU_RUN -> unconnected-(U82-Q_N-Pad3)
- U82 pad 6: unconnected-(U82-Q_N-Pad6) -> FINAL_PROOF_CLEAR_N
- U90 pad 2: CTRL_RAIL_OK_LOCAL -> RUNTIME_HEALTHY
- U92 pad 4: SUP_RUN_OK_LOCAL -> PRE_ISO_RUN_OK
Routing:
- net COIL_RET: track 0.00 -> 660.9 mm, vias 0 -> 4
- net AUX_24V: track 398.2 -> 1006.5 mm, vias 5 -> 6
- net ADMIT: track 0.00 -> 325.2 mm, vias 0 -> 6
- net SOURCE_DRIVE_TIMED: track 0.00 -> 290.1 mm, vias 0 -> 4
- net KPA_FB_EXC: track 0.00 -> 251.2 mm, vias 0 -> 7
- net FINAL_PROOF_CLEAR_N: track 0.00 -> 230.1 mm, vias 0 -> 6
- net KPA_MIRROR: track 0.00 -> 228.5 mm, vias 0 -> 5
- net KPB_MIRROR: track 0.00 -> 224.6 mm, vias 0 -> 6
- net KPB_FB_EXC: track 0.00 -> 224.0 mm, vias 0 -> 6
- net CMD_KPB: track 0.00 -> 217.9 mm, vias 0 -> 4
- net CMD_KPA: track 0.00 -> 214.4 mm, vias 0 -> 5
- net BUDGET_OR_PROOF: track 18.8 -> 229.0 mm, vias 2 -> 5
- net POD_5V: track 331.5 -> 538.9 mm, vias 3 -> 6
- net K1_MIRROR_24V: track 0.00 -> 206.3 mm, vias 0 -> 1
- net K2_MIRROR_24V: track 0.00 -> 200.5 mm, vias 0 -> 1
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- added copper zone on B.Cu, net AUX_0V
- added copper zone on In1.Cu, net AUX_0V
- added copper zone on In1.Cu, net COIL_RET
- added copper zone on F.Cu, net K1_SUB
- added copper zone on F.Cu, net K2_SUB
- added copper zone on F.Cu, net KB_SUB
- added copper zone on F.Cu, net KPA_SUB
- added copper zone on F.Cu, net KPB_SUB
- added copper zone on F.Cu, net POD_3V3
