File: zapote/power-stage-120v/prototype-closure/round5/boards/central/native/supervisor.kicad_sch (KiCad schematic)
At the start: 0 parts

Commit message: WIP snapshot of worktrees/mit-product-guidance (2026-10-08)
Uncommitted Codex prototype-closure work (round5 boards, round6
investigation, firmware power adapter), snapshotted without touching the
worktree. Raw solver output under output/temper-prototype-closure/ is
not included.

Co-Authored-By: Claude Opus 5.5 (1M context) <noreply@anthropic.com>
Other:
- added sheet FEEDBACK_2 (FEEDBACK_2.kicad_sch)
- added sheet FEEDBACK_3 (FEEDBACK_3.kicad_sch)
- added sheet FEEDBACK_4 (FEEDBACK_4.kicad_sch)
- added sheet FEEDBACK_5 (FEEDBACK_5.kicad_sch)
- added sheet FEEDBACK_6 (FEEDBACK_6.kicad_sch)
- added sheet FEEDBACK_7 (FEEDBACK_7.kicad_sch)
- added sheet FEEDBACK_8 (FEEDBACK_8.kicad_sch)
- added sheet FEEDBACK_9 (FEEDBACK_9.kicad_sch)
- added sheet HARDWARE_14 (HARDWARE_14.kicad_sch)
- added sheet HARDWARE_15 (HARDWARE_15.kicad_sch)
- added sheet HARDWARE_16 (HARDWARE_16.kicad_sch)
- added sheet HARDWARE_17 (HARDWARE_17.kicad_sch)
- added sheet POWER_2 (POWER_2.kicad_sch)
