File: zapote/power-stage-120v/prototype-closure/round5/boards/native/pre-sensor/pre-sensor.kicad_sch (KiCad schematic)
At the start: 17 parts, among them J1 HV leads, J2 B6B-XH-A, U1 AMC3330DWE

Commit message: WIP snapshot of worktrees/mit-product-guidance (2026-10-08)
Uncommitted Codex prototype-closure work (round5 boards, round6
investigation, firmware power adapter), snapshotted without touching the
worktree. Raw solver output under output/temper-prototype-closure/ is
not included.

Co-Authored-By: Claude Opus 5.5 (1M context) <noreply@anthropic.com>
Parts:
- added R10: 10kR, Resistor_SMD:R_0603_1608Metric, symbol Sensor:R_Small_US
- added R7, R8: 249kR 0.1%, Resistor_SMD:R_1206_3216Metric, symbol Sensor:R_Small_US
- added R9: 2.49kR 0.1%, Resistor_SMD:R_1206_3216Metric, symbol Sensor:R_Small_US
- R5: value 4.02kR 0.1% -> 249kR 0.1%; MPN TNPW12064K02BEEA 4.02kR 0.1% -> TNPW1206249KBEEA 249kR 0.1%
- R6: value 10kR -> 249kR 0.1%; footprint Resistor_SMD:R_0603_1608Metric -> Resistor_SMD:R_1206_3216Metric; MPN 10kR CRCW060310K0FKEA -> TNPW1206249KBEEA 249kR 0.1%
Connections:
- net L_PRE: now also R9.2; no longer R5.2
- net POD_3V3: now also R10.1; no longer R6.1
- net VPRE_DIAG_N: now also R10.2; no longer R6.2
- net VPRE_TAP: now also R8.2, R9.1; no longer R4.2, R5.1
- new net VPRE_DIV3: R4.2, R5.1
- new net VPRE_DIV4: R5.2, R6.1
- new net VPRE_DIV5: R6.2, R7.1
- new net VPRE_DIV6: R7.2, R8.1
Other:
- moved on the sheet: R2, R3, R4, R5, R6
