File: instruments/differential-probe/cad/differential-probe.kicad_sch (KiCad schematic)
At the start: 54 parts, among them U1 ADA4817-1ARDZ-R7, U2 ADA4817-1ARDZ-R7

Commit message: fix(instruments): compact the probe and keep range switching outside feedback
Add fine compensation trimmers, fixed OPA810 gain stages and conservative
initial-envelope warning thresholds with analog-offset allowances. Reduce
the PCB to 240 x 84 mm using the simultaneous 3 kV input envelope, retaining
matched divider geometry, slots and explicit spacing rules.

Regenerate native schematic, BOM, routed PCB and validation artifacts.
Document manufacturer-model limits, bench qualification and the corrected
stage-53 CT calculations without changing the pinned power-stage board.
Parts:
- added CT1, CT2: 12-60 pF / set ~35 pF, Probe:GKG60015_TopAdjust, symbol Probe:C_Trim
- C45, C55: value 82 pF -> 47 pF; MPN C0805C820J5GACTU -> C0805C470J5GACTU
Connections:
- net GND: now also CT1.2, CT2.2
- net TAP_N: now also CT2.1
- net TAP_P: now also CT1.1
Other:
- note added: "AC COMPENSATION / coarse C0G bank + accessible fine trim"
- note added: "Coarse Csum = 13.158 nF per leg. CT1/2: rotor to GND; nominal 35.4 pF. Adjust through shield tool holes. Select coarse bank after assembly. TIP_P / TIP_N: captive HV leads."
- note removed: "AC COMPENSATION / C0G selection pads; trim with shield fitted"
- note removed: "Starting Csum = 13.193 nF per leg. Select on the bench. Do not assume nominal values deliver 60 dB CMRR. Local decoupling for U1/U2 is on the power sheet. TIP_P / TIP_N: captive HV leads, no SMA inputs."
