File: instruments/differential-probe/cad/differential-probe.kicad_sch (KiCad schematic)
At the start: 56 parts, among them U1 ADA4817-1ARDZ-R7, U2 ADA4817-1ARDZ-R7

Commit message: wip(instruments): Rev C mirrored HV ladder layout, TL431-free warning, OPA2810 chain
Co-Authored-By: Claude Opus 5.5 <noreply@anthropic.com>
Parts:
- removed C44, C54: 220 pF, Capacitor_SMD:C_0805_2012Metric, symbol Probe:C
- removed C45, C55: 47 pF, Capacitor_SMD:C_0805_2012Metric, symbol Probe:C
- removed C46, C56: 10 pF, Capacitor_SMD:C_0805_2012Metric, symbol Probe:C
- removed C47, C57: 1 pF, Capacitor_SMD:C_0805_2012Metric, symbol Probe:C
- removed R10, R26, R27, R28, R29, R30, R6, R7, R8, R9: 1 MR / 0.1%, Resistor_SMD:R_2512_6332Metric, symbol Probe:R_Small_US
- removed U2: ADA4817-1ARDZ-R7, Probe:ADA4817_RD-8-4, symbol Probe:ADA4817
- C42, C52: value 2.2 nF -> SOT 3.0 nF / 1%; MPN C0805C222J5GACTU -> C0805C302F5GACTU
- C43, C53: value 680 pF -> SOT 160 pF / 1%; MPN C0805C681J5GACTU -> C0805C161F5GACTU
- CT1, CT2: value 12-60 pF / set ~35 pF -> 12-60 pF / set ~33 pF
- R1, R2, R21, R22, R23, R24, R25, R3, R4, R5: value 1 MR / 0.1% -> 2 MR / 0.1%; MPN HVCB2512BDE1M00 -> HVCB2512BDE2M00
- R12, R32: MPN RT0805BRD07220L -> RT0805BRD07220RL
- U1: value ADA4817-1ARDZ-R7 -> OPA2810IDR; footprint Probe:ADA4817_RD-8-4 -> Package_SO:SOIC-8_3.9x4.9mm_P1.27mm; symbol Probe:ADA4817 -> Probe:OPA2810; LCSC C207502 -> C1849413; MPN ADA4817-1ARDZ-R7 -> OPA2810IDR; Manufacturer Analog Devices -> Texas Instruments
Connections:
- net REF_N is gone; now on net -4V8: D1.1 (A1), D2.1 (A1)
- net REF_P is gone; now on net +4V8: D1.2 (K2), D2.2 (K2)
- net +4V8: no longer U1.7 (+VS)
- net BUF_N: now also U1.6 (-IN2), U1.7 (OUT2)
- net BUF_P: no longer U1.6 (OUT)
- net GND: no longer U1.9 (EP)
- net IN_N: now also U1.5 (+IN2)
- net TAP_N: now also R25.2
- net TAP_P: now also R5.2
- net P_SEG1: now reaches C1.2, C2.1
- net P_SEG1: now also R1.2, R2.1; no longer R2.2, R3.1
- net P_SEG2: now reaches C2.2, C3.1
- net P_SEG2: now also R2.2, R3.1; no longer R4.2, R5.1
- net P_SEG3: now reaches C3.2, C4.1
- net P_SEG3: now also R3.2, R4.1
- net P_SEG4: now reaches C4.2, C5.1
- net P_SEG4: now also R4.2, R5.1
- net N_SEG1: now reaches C21.2, C22.1
- net N_SEG1: now also R21.2, R22.1; no longer R22.2, R23.1
- net N_SEG2: now reaches C22.2, C23.1
- net N_SEG2: now also R22.2, R23.1; no longer R24.2, R25.1
- net N_SEG3: now reaches C23.2, C24.1
- net N_SEG3: now also R23.2, R24.1
- net N_SEG4: now reaches C24.2, C25.1
- net N_SEG4: now also R24.2, R25.1
- net TRIM_P: now reaches R11.2, RV1.1 (CCW)
- net TRIM_N: now reaches R31.2, RV2.1 (CCW)
- no-connect marks 2 -> 0
Other:
- note added: "2000:1 INPUTS / mirror-matched geometry about the inter-leg slot, fixed grounded shield"
- note added: "AC COMPENSATION / fixed C0G + two select-on-test C0G + accessible fine trim"
- note added: "Fixed 10 nF 1% + select-on-test S1 (E24 1.6-3.9 nF, 1%) + S2 (E24 0-360 pF, 1%) + 12-60 pF trimmer. Nominal 10 nF + 3.0 nF + 160 pF + ~33 pF. CT1/2: rotor to GND. Adjust through shield tool holes. TIP_P / TIP_N: captive HV leads."
- note removed: "2000:1 INPUTS / matched geometry, fixed grounded shield"
- note removed: "AC COMPENSATION / coarse C0G bank + accessible fine trim"
- note removed: "Coarse Csum = 13.158 nF per leg. CT1/2: rotor to GND; nominal 35.4 pF. Adjust through shield tool holes. Select coarse bank after assembly. TIP_P / TIP_N: captive HV leads."
- moved on the sheet: R1, R2, R21, R22, R23, R24, R25, R3, R4, R5

Commit message: feat(probe): Rev C cost-down: HV12 divider, Yageo C0G, E-Switch toggles, Basic parts
Implements docs/cost-down.md with no layout change (pads, tracks and
courtyards identical to 5b9a9530b):

- HV divider: Uni-Royal HV121WF2004T4E (1 %, 1 W, 3 kV, JLC-stocked)
  replaces Stackpole HVCB2512BDE2M00; DC trim becomes 4.87 k 0.1 % +
  500 ohm (covers 1 % and 0.1 % strings, so HVCB stays a drop-in).
- Yageo CC1812JKNPOEBN330 (33 pF 3 kV NP0) and CC1206FKNPO9BN103
  (10 nF 1 % NP0) replace the KEMET parts.
- E-Switch 100SP1T1B5M7RE / 100DP1T1B1M7QEH replace the C&K toggles;
  footprints renamed ESwitch_100_M7_* from the E-Switch M7 drawing.
- Non-precision positions move to JLC Basic parts; C61 and the 10 uF
  move to stocked equivalents. Extended MPNs placed by JLC: 33 -> 24.
- check.rs: new MPN asserts, 1 %-string trim proof, divider TCR drift,
  1 W rating text with the 2+3 split fault case stated.

Two boards: components $535.81 -> $148.63 (ledger); with JLC fees,
PCB, ~$100 leads and enclosures $866.44 -> $448.20 (validation/cost.txt).

Co-Authored-By: Claude Opus 5.5 <noreply@anthropic.com>
Parts:
- C1, C2, C21, C22, C23, C24, C25, C3, C4, C5: LCSC (none) -> C2359543; MPN C1812C330JHGACTU -> CC1812JKNPOEBN330; Manufacturer KEMET -> Yageo
- C41, C51: LCSC (none) -> C541597; MPN C1206C103F5GACTU -> CC1206FKNPO9BN103; Manufacturer KEMET -> Yageo
- R1, R2, R21, R22, R23, R24, R25, R3, R4, R5: value 2 MR / 0.1% -> 2 MR / 1% / 3 kV; LCSC (none) -> C2779442; MPN HVCB2512BDE2M00 -> HV121WF2004T4E; Manufacturer Stackpole -> Uni-Royal
- R11, R31: value 4.99 kR / 0.01% -> 4.87 kR / 0.1%; LCSC C3942722 -> C861446; MPN RNCF0603TKY4K99 -> RT0603BRD074K87L; Manufacturer Stackpole -> Yageo
- R12, R32: LCSC (none) -> C17557; MPN RT0805BRD07220RL -> 0805W8F2200T5E; Manufacturer Yageo -> Uni-Royal
- RV1, RV2: value 50 R / set 12.50 R -> 500 R / set 132.5 R; LCSC C83692 -> C69564; MPN 3296W-1-500LF -> 3296W-1-501LF
