File: instruments/lcr-meter/cad/adc.kicad_sch (KiCad schematic)
At the start: 41 parts, among them U10 ADS9224RIRHBR, U8 THS4551IRGTR, U9 THS4551IRGTR

Commit message: lcr-meter Rev D: apply Tier 1 audit fixes
Hand-routed layout edits (cad/tools/edit_lib.py, no autorouter):
- Vias in every exposed pad: U1 8, U8/U9/U10 5, U11/U12 6 (were 0), U13 9.
- ADS9224R: 10 uF X7R 0805 reference caps at 1.56 mm, REFM joined to the
  cap before its via; 1 uF AVDD caps at 1.67/2.46 mm from pins 12/29.
- TPS7A4901/TPS7A3001: support parts packed per TI layout; FB nodes
  13.2/12.0 -> 5.2/5.3 mm, NR 2.1 mm. LDOIN_N In2 run moved off the pads.
- TPS65131 dividers compacted: CONV_FBP 13.1 -> 9.1 mm, CONV_FBN 16.8 -> 12.3 mm.
- RP2040: 1 uF at VREG_VIN (C5).

Parts: red status LED, basic ferrites, W25Q128JV flash (stock), C84,
CL32B106KBJNNNE on the 14 V and converter-input caps, C18/C103 basic,
C36 1 uF -> 100 nF. Extended lines 34 -> 30.

Firmware: settle max(150 ms, 20 cycles); BOOT -> reset_usb_boot().
Host 0.7.0: `temper-lcr boot PORT`.

Withdrawn after checking: converter dividers to TI example values (VPOS
15.105 V at the tolerance stack), 1 % LDO dividers (U12 headroom 0.74 V),
SRV05-4 (pinout unverifiable). regulator_check.py now reads design.json
instead of stale Rev C values.

DRC 0, unconnected 0, parity 0, ERC 0; independent check 576 pins, 0
findings; host 29 tests pass.

Co-Authored-By: Claude Opus 5.5 <noreply@anthropic.com>
Parts:
- C72, C73: value 22uF 25V -> 10uF 16V X7R; footprint LCR:C_1210_3225Metric -> LCR:C_0805_2012Metric; LCSC C21397 -> C95841; MPN GRM32ER71E226KE15L -> CL21B106KOQNNNE; Manufacturer Murata Electronics -> Samsung Electro-Mechanics; Unit_USD 0.4151 -> 0.12
- C76, C77: value 1uF 50V -> 1uF 50V X5R; footprint LCR:C_0805_2012Metric -> LCR:C_0603_1608Metric; LCSC C28323 -> C15849; MPN CL21B105KBFNNNE -> CL10A105KB8NNNC; Unit_USD 0.0344 -> 0.0153
